File: schematics/supply/supply.kicad_pcb (KiCad board)
At the start: 4 copper layers, 237.5 x 175 mm, 307 parts, among them J1 Conn_01x02_Pin, J11 Conn_01x04_Pin, J13 USBASP, J14 USBASP, J15 Conn_01x06_Pin, J17 banana jack + fuse 15A, J18 banana jack + fuse 15A, J19 Conn_02x04_Odd_Even, J2 Conn_01x02_Pin, J20 jst xh angle, J21 jst xh angle, J3 Conn_01x01_Pin, J4 Conn_01x01_Pin, J5 CW2B-10A-T, J6 USB_A, J7 USB_A, J8 USB_A, J9 Conn_01x04_Pin, K1 SRD-12VDC-SL-C, M1 Fan, Q1 STP13NK60Z, Q10 IRLML0030, Q11 IRLML0030, Q12 IRLML0030, Q13 IRLML5203, Q14 IRLML5203, Q2 IRLML5203, Q3 40N06, Q4 STP13NK60Z, Q5 STP13NK60Z, Q6 IRLML0030, Q7 IRLML5203, Q8 IRLML5203, Q9 IRLML0030, SW3 SW_Push, U1 ICE2PCS01, U10 IRS2153S, U11 LM158DR, U12 IP2163, U13 LM158DR, U14 TL432DBZ, U15 LM158DR, U16 LM1085-3.3, U17 ATmega328-A, U18 ATtiny1616-M, U2 TL331, U20 LM158DR, U21 EL817, U22 IRS2153S, U23 TL331, U24 INA169, U25 INA3221, U3 R7731, U4 EL817, U5 TL432DBZ, U6 INA3221, U7 EL817, U8 MC34063AD, U9 L78L33ACUTR, X1 HC-49U, 16MHz, X2 CSX-750FCC, 16MHz, Y1 B32022A3223M000

Commit message: Board prepared to order
Parts:
- F1: value 10x38, 4A with fuseholder -> C10G4 with fuseholder
- L4: value SPM6550T-2R2M -> SPM6550T-R68M
- moved C62 6.25 mm to (148.0, 72.3)
- moved TP4 5.90 mm to (128.9, 62.8)
- moved U24 5.64 mm to (147.8, 72.2)
- moved R70 5.56 mm to (142.8, 72.5), turned to -90 degrees
- moved C57 5.45 mm to (136.2, 68.2)
- moved R69 5.45 mm to (147.7, 68.0)
- moved J18 3.47 mm to (154.3, 68.5)
- moved H2 2.78 mm to (163.0, 64.6)
- moved R59 2.75 mm to (161.0, 73.0)
- moved CLR6 2.28 mm to (109.9, 88.8)
- moved Q10 1.75 mm to (161.0, 77.3)
- moved TR4 1.69 mm to (154.6, 111.5)
- moved L1 1.39 mm to (286.5, 110.4)
- moved D27 1.30 mm to (114.6, 94.5)
- moved C55 0.83 mm to (189.8, 104.9)
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Routing:
- net Net-(U24-+): track 130.7 -> 152.3 mm
- net /Control & Fan/+5V_VSYS: track 701.1 -> 718.8 mm
- net GND: track 922.4 -> 929.6 mm
- net /Control & Fan/POWER_OUTPUT_CURRENT_SENSE: track 60.1 -> 65.2 mm
- net /Control & Fan/POWER_OUTPUT_FB: track 72.3 -> 76.4 mm
- net Net-(R59-Pad2): track 6.66 -> 4.00 mm
- net Net-(D27-K): track 48.4 -> 50.5 mm
- net /Output connectors/POWER_OUT: track 13.4 -> 11.3 mm
- net Net-(Q10-D): track 5.00 -> 3.23 mm
- net Net-(D6-A): track 67.9 -> 66.5 mm
- net Net-(C55-Pad1): track 28.2 -> 26.8 mm
- net Net-(D27-A-Pad3): track 156.2 -> 155.3 mm
- net Net-(D4-K): track 31.5 -> 30.8 mm
- net Net-(D27-A-Pad1): track 100.9 -> 100.1 mm
- net /Power output/RC_SNABBER_MIDDLEPOINT: track 102.8 -> 103.4 mm
Other:
- board text added: "Supply board#1 v1.0"
- board text added: "Supply board#2 v1.0"
- board text removed: "Supply part1 v1.0"
- board text removed: "Supply part2 v1.0"

Commit message: Created gerber-files to check order cost
Parts:
- moved C1 13.6 mm to (206.7, 109.8)
- moved C10 13.6 mm to (262.7, 136.1)
- moved C11 13.6 mm to (258.9, 128.8)
- moved C2 13.6 mm to (233.6, 162.9)
- moved C3 13.6 mm to (291.9, 160.3)
- moved C4 13.6 mm to (269.4, 136.6)
- moved C5 13.6 mm to (306.9, 137.8)
- moved C6 13.6 mm to (280.2, 151.3)
- moved C8 13.6 mm to (270.9, 112.6)
- moved C9 13.6 mm to (290.8, 121.2)
- moved CLR1 13.6 mm to (221.4, 91.8)
- moved CLR2 13.6 mm to (227.5, 155.4)
- moved CP1 13.6 mm to (233.8, 113.8)
- moved CP5 13.6 mm to (207.4, 137.9)
- moved D1 13.6 mm to (213.7, 94.3)
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Other:
- board size 237.5 x 175 mm -> 224 x 175 mm
