File: schematics/supply/supply.kicad_pcb (KiCad board)
At the start: 4 copper layers, 110 x 179.8 mm, 250 parts, among them J1 Conn_01x02_Pin, J10 USBASP, J12 JST XH B3B, J13 Conn_01x06_Pin, J16 Conn_01x05_Pin, J17 banana jack + fuse 15A, J18 banana jack + fuse 15A, J2 Conn_01x01_Pin, J22 Conn_02x04_Odd_Even, J23 jst xh angle, J24 jst xh angle, J25 Conn_01x05_Socket, J3 USB_A, J4 USB_A, J5 USB_A, J6 Conn_01x04_Pin, J8 Conn_01x04_Pin, M1 Fan, Q1 STP13NK60Z, Q10 STP13NK60Z, Q11 STP13NK60Z, Q12 IRLML0030, Q13 IRF7425PbF, Q14 IRF7425PbF, Q2 STP13NK60Z, Q3 IRLML0030, Q4 IRLML0030, Q5 IRLML5203, Q6 IRLML0030, Q7 IRLML0030, Q8 IRLML0030, Q9 IRLML0030, SW3 SW_Push, U1 INA3221, U10 LM158DR, U11 LM158DR, U12 TL432DBZ, U13 LM1085-3.3, U14 ATmega328-A, U15 ATtiny1616-M, U17 AD9833xRM, U18 MCP4726A0T-E/CH, U19 MAX961, U2 XL6009, U20 LM158DR, U21 FAN3100, U22 EL817, U23 EL817, U24 UC3525, U25 IR2117, U26 IR2117, U27 INA169, U28 TP4056, U29 INA3221, U3 EL817, U4 L78L33ACUTR, U5 UC3525, U6 LM158DR, U7 IP2163, U8 IR2117, U9 IR2117, X1 HC-49U, 16MHz, X2 ???

Commit message: re-design supply board
Parts:
- removed J25: Conn_01x05_Socket, Connector_PinHeader_2.54mm:PinHeader_1x05_P2.54mm_Vertical
- added C41: 10 nF, Capacitor_SMD:C_0603_1608Metric, B.Cu at (96.0, 163.1)
- added J15: USBASP, Connector_PinHeader_2.54mm:PinHeader_2x05_P2.54mm_Vertical, F.Cu at (88.8, 85.7)
- added J2: RFShield_OnePiece, Library:EMI_SHIELD_1P_2H, F.Cu at (124.0, 88.7)
- added J3: RFShield_OnePiece, Library:EMI_SHIELD_1P_2H, F.Cu at (89.0, 171.7)
- added J5: RFShield_OnePiece, Library:EMI_SHIELD_1P_2H, F.Cu at (124.0, 105.7)
- added J6: RFShield_OnePiece, Library:EMI_SHIELD_1P_2H, F.Cu at (124.0, 147.7)
- added R40: 10K, Resistor_SMD:R_0805_2012Metric, F.Cu at (104.6, 153.2)
- added R41: 10K, Resistor_SMD:R_0805_2012Metric, F.Cu at (101.8, 152.4)
- added R42: 10K, Resistor_SMD:R_0805_2012Metric, F.Cu at (106.0, 161.9)
- added TP1: 5V_A, TestPoint:TestPoint_Pad_1.0x1.0mm, F.Cu at (165.8, 183.7)
- added TP10: F_R1, TestPoint:TestPoint_Pad_1.0x1.0mm, F.Cu at (92.3, 111.6)
- added TP11: F_R2, TestPoint:TestPoint_Pad_1.0x1.0mm, F.Cu at (96.6, 111.6)
- added TP12: F_EN, TestPoint:TestPoint_Pad_1.0x1.0mm, F.Cu at (96.6, 101.9)
- added TP13: BTN_FB, TestPoint:TestPoint_Pad_1.0x1.0mm, F.Cu at (117.9, 109.5)
- added TP14: IC_FB, TestPoint:TestPoint_Pad_1.0x1.0mm, F.Cu at (117.9, 107.1)
- added TP15: SGN, TestPoint:TestPoint_Pad_1.0x1.0mm, F.Cu at (111.0, 174.2)
- added TP16: PW_FB, TestPoint:TestPoint_Pad_1.0x1.0mm, F.Cu at (119.2, 95.5)
- added TP17: PW_A, TestPoint:TestPoint_Pad_1.0x1.0mm, B.Cu at (155.7, 119.9)
- added TP18: PW_B, TestPoint:TestPoint_Pad_1.0x1.0mm, B.Cu at (151.0, 120.0)
- added TP2: 5V_B, TestPoint:TestPoint_Pad_1.0x1.0mm, F.Cu at (154.8, 182.8)
- added TP4: PW_CS, TestPoint:TestPoint_Pad_1.0x1.0mm, F.Cu at (94.1, 78.6)
- added TP5: PW_VS, TestPoint:TestPoint_Pad_1.0x1.0mm, F.Cu at (93.9, 82.1)
- added TP6: PW_SHDN#, TestPoint:TestPoint_Pad_1.0x1.0mm, F.Cu at (104.6, 92.7)
- added TP7: SGN_DAC, TestPoint:TestPoint_Pad_1.0x1.0mm, F.Cu at (96.9, 161.1)
- added TP8: SGN_GEN, TestPoint:TestPoint_Pad_1.0x1.0mm, F.Cu at (100.6, 160.7)
- added TP9: F_IC, TestPoint:TestPoint_Pad_1.0x1.0mm, F.Cu at (94.5, 111.6)
- RV2: moved to F.Cu
- U10, U11, U6: footprint Package_SO:SOP-8_5.28x5.23mm_P1.27mm -> Package_SO:SOP-8_3.76x4.96mm_P1.27mm
- moved H4 64.2 mm to (90.5, 154.5)
- moved R1 5.60 mm to (124.5, 190.2)
- moved L1 5.09 mm to (100.5, 182.2)
- moved R30 4.20 mm to (94.6, 94.4)
- moved TR1 3.28 mm to (182.9, 171.2)
- moved R53 3.10 mm to (162.0, 85.9)
- moved C6 2.48 mm to (104.3, 221.4)
- moved U4 2.48 mm to (100.8, 220.2)
- moved C36 2.43 mm to (94.9, 122.3)
- moved C2 2.21 mm to (98.6, 175.5), turned to -90 degrees
- moved TP3 2.20 mm to (90.0, 103.2)
- moved H3 2.00 mm to (103.5, 81.0)
- moved NT1 1.80 mm to (109.5, 182.2)
- moved RV1 1.60 mm to (115.5, 203.2)
- moved R22 1.53 mm to (161.9, 227.7), turned to 90 degrees
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- renumbered C13 to C11, C14 to C12, C15 to C13, C16 to C14, C17 to C15, C18 to C16, C19 to C17, C20 to C18, C21 to C19, C22 to C20, C23 to C21, C24 to C22, C25 to C23, C26 to C24, C27 to C25, C28 to C26, C29 to C27, C30 to C28, C31 to C29, C32 to C30, C33 to C31, C34 to C32, C35 to C33, C36 to C34, C38 to C35, C39 to C36, C40 to C37, C41 to C38, C42 to C39, C43 to C40, C44 to C42, C45 to C43, C46 to C44, C47 to C45, C48 to C46, C49 to C47, C50 to C48, C51 to C49, C52 to C50, C53 to C51, C54 to C52, C55 to C53, C58 to C54, C59 to C55, C60 to C56, C61 to C57, C62 to C58, C69 to C59, C63 to C60, C64 to C61, C65 to C62, C66 to C63, C67 to C64, C68 to C65, J6 to J10, J8 to J12, J10 to J14, J12 to J16, J13 to J17, J16 to J20, J17 to J21, J18 to J22, J22 to J26, J23 to J27, J24 to J28, J2 to J4, J3 to J7, J4 to J8, J5 to J9, R40 to R43, R41 to R44, R42 to R45, R43 to R46, R44 to R47, R45 to R48, R46 to R49, R47 to R50, R48 to R51, R49 to R52, R50 to R53, R51 to R54, R52 to R55, R53 to R56, R54 to R57, R55 to R58, R56 to R59, R57 to R60, R58 to R61, R59 to R62, R60 to R63, R61 to R64, R62 to R65, R63 to R66, R64 to R67, R65 to R68, R66 to R69, R67 to R70, TP1 to TP3
Connections:
- D10 pad 1: GND -> /Internal 5V & out usb/+5V_OUT
- D10 pad 2: /Internal 5V & out usb/+5V_OUT -> GND
- D11 pad 1: GND -> /Control & Fan/+5V_VSYS
- D11 pad 2: /Control & Fan/+5V_VSYS -> GND
- D4 pad 1: GND -> /Internal 5V & out usb/VBUS_1
- D4 pad 2: /Internal 5V & out usb/VBUS_1 -> GND
Routing:
- net GNDPWR: track 457.9 -> 538.8 mm
- net GND: track 591.0 -> 546.7 mm, vias 23 -> 25
- net Net-(D8-A-Pad1): track 90.0 -> 104.0 mm
- net /Power output/RC_SNABBER_MIDDLEPOINT: track 93.9 -> 102.7 mm, vias 0 -> 1
- net Net-(U5-OUTA): track 5.15 -> 13.6 mm, vias 1 -> 2
- net /Control & Fan/IS_ONOFF_BUTTON_PRESSED: track 55.9 -> 63.5 mm
- net /Internal 5V & out usb/VREF_2V5: track 115.9 -> 108.8 mm
- net /Control & Fan/+5V_VSYS: track 640.2 -> 633.2 mm, vias 14 -> 21
- net /Internal 5V & out usb/VBUS_1: track 49.6 -> 56.4 mm, vias 3 -> 2
- net /Internal 5V & out usb/RC_SNABBER_MIDDLEPOINT: track 62.9 -> 69.3 mm
- net /Control & Fan/ATTINY_RESET#: track 12.4 -> 18.2 mm
- net Net-(R1-Pad1): track 2.01 -> 7.41 mm
- net Net-(D1-A): track 20.5 -> 25.8 mm
- net Net-(U2-FB): track 40.4 -> 45.2 mm
- net /Control & Fan/POWER_OUTPUT_SHUTDOWN#: track 69.6 -> 74.0 mm, vias 2 -> 3
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Other:
- board text removed: "-"
- board text removed: "GND"
- board text removed: "PWOUT GND"
- board text removed: "[I]"
- board text removed: "[V]"
