File: schematics/supply/output_5v_usb.kicad_sch (KiCad schematic)
At the start: 89 parts, among them J2 USB_A, Q3 40N06, U10 IRS2153S, U11 LM158DR, U12 IP2163, U13 LM158DR, U14 TL432DBZ, U15 LM158DR, U16 LM1085-3.3, U2 EL817, U6 INA3221, U8 MC34063AD, U9 L78L33ACUTR

Commit message: Some changes in board - Im preparing it to production
Parts:
- removed F2: JK30-300, Capacitor_THT:C_Disc_D11.0mm_W5.0mm_P5.00mm, symbol Device:Polyfuse
- removed F3, F4: JK30-200, Capacitor_THT:C_Disc_D11.0mm_W5.0mm_P5.00mm, symbol Device:Polyfuse
- added F2: 5A, Connector_Wire:SolderWire-0.75sqmm_1x02_P4.8mm_D1.25mm_OD2.3mm, symbol Device:Fuse
- added F3, F4: 3A, Connector_Wire:SolderWire-0.75sqmm_1x02_P4.8mm_D1.25mm_OD2.3mm, symbol Device:Fuse
Connections:
- net USB_1_BP: now also F2.1
- net USB_2_+5V: now also F3.1
- net USB_3_+5V: now also F4.1
- net VBUS_1_+: now also F2.2
- net VBUS_2_+: now also F3.2
- net VBUS_3_+: now also F4.2
Changed lines of the file:
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@@
-    )
-  )
-  (symbol (lib_id "Device:Polyfuse") (at 152.4 142.24 90) (unit 1)
-    (in_bom yes) (on_board yes) (dnp no) (fields_autoplaced)
-    (property "Reference" "F2" (at 152.4 137.16 90)
-      (effects (font (size 1.27 1.27)))
-    )
-    (property "Value" "JK30-300" (at 152.4 139.7 90)
-      (effects (font (size 1.27 1.27)))
-    )
-    (property "Footprint" "Capacitor_THT:C_Disc_D11.0mm_W5.0mm_P5.00mm" (at 157.48 140.97 0)
-      (effects (font (size 1.27 1.27)) (justify left) hide)
-    )
-    (property "Datasheet" "~" (at 152.4 142.24 0)
-      (effects (font (size 1.27 1.27)) hide)
-    )
-    (pin "1")
-    (pin "2")
-    (instances
-      (project "supply"
-        (path "/1e139717-fcd1-4008-a6ea-4c993845e928/bcabd54f-a555-4409-9a4f-89c20a3d7682"
-          (reference "F2") (unit 1)
-        )
-      )
     )
   )
@@
         (path "/1e139717-fcd1-4008-a6ea-4c993845e928/bcabd54f-a555-4409-9a4f-89c20a3d7682"
           (reference "R42") (unit 1)
+        )
+      )
+    )
+  )
+  (symbol (lib_id "Device:Fuse") (at 226.06 142.24 90) (unit 1)
+    (in_bom yes) (on_board yes) (dnp no) (fields_autoplaced)
+    (property "Reference" "F3" (at 226.06 137.16 90)
+      (effects (font (size 1.27 1.27)))
+    )
+    (property "Value" "3A" (at 226.06 139.7 90)
+      (effects (font (size 1.27 1.27)))
+    )
+    (property "Footprint" "Connector_Wire:SolderWire-0.75sqmm_1x02_P4.8mm_D1.25mm_OD2.3mm" (at 226.06 144.018 90)
+      (effects (font (size 1.27 1.27)) hide)
+    )
+    (property "Datasheet" "~" (at 226.06 142.24 0)
+      (effects (font (size 1.27 1.27)) hide)
+    )
+    (pin "1")
+    (pin "2")
+    (instances
+      (project "supply"
+        (path "/1e139717-fcd1-4008-a6ea-4c993845e928/bcabd54f-a555-4409-9a4f-89c20a3d7682"
+          (reference "F3") (unit 1)
         )
       )
@@
         (path "/1e139717-fcd1-4008-a6ea-4c993845e928/bcabd54f-a555-4409-9a4f-89c20a3d7682"
           (reference "J8") (unit 1)
+        )
+      )
+    )
+  )
+  (symbol (lib_id "Device:Fuse") (at 302.26 140.97 90) (unit 1)
+    (in_bom yes) (on_board yes) (dnp no) (fields_autoplaced)
+    (property "Reference" "F4" (at 302.26 135.89 90)
+      (effects (font (size 1.27 1.27)))
+    )
+    (property "Value" "3A" (at 302.26 138.43 90)
+      (effects (font (size 1.27 1.27)))
+    )
+    (property "Footprint" "Connector_Wire:SolderWire-0.75sqmm_1x02_P4.8mm_D1.25mm_OD2.3mm" (at 302.26 142.748 90)
+      (effects (font (size 1.27 1.27)) hide)
+    )
+    (property "Datasheet" "~" (at 302.26 140.97 0)
+      (effects (font (size 1.27 1.27)) hide)
+    )
+    (pin "1")
+    (pin "2")
+    (instances
+      (project "supply"
+        (path "/1e139717-fcd1-4008-a6ea-4c993845e928/bcabd54f-a555-4409-9a4f-89c20a3d7682"
+          (reference "F4") (unit 1)
         )
       )
@@
     )
   )
-  (symbol (lib_id "Device:Polyfuse") (at 302.26 140.97 90) (unit 1)
-    (in_bom yes) (on_board yes) (dnp no) (fields_autoplaced)
-    (property "Reference" "F4" (at 302.26 135.89 90)
-      (effects (font (size 1.27 1.27)))
-    )
-    (property "Value" "JK30-200" (at 302.26 138.43 90)
-      (effects (font (size 1.27 1.27)))
-    )
-    (property "Footprint" "Capacitor_THT:C_Disc_D11.0mm_W5.0mm_P5.00mm" (at 307.34 139.7 0)
-      (effects (font (size 1.27 1.27)) (justify left) hide)
-    )
-    (property "Datasheet" "~" (at 302.26 140.97 0)
-      (effects (font (size 1.27 1.27)) hide)
-    )
-    (pin "1")
-    (pin "2")
-    (instances
-      (project "supply"
-        (path "/1e139717-fcd1-4008-a6ea-4c993845e928/bcabd54f-a555-4409-9a4f-89c20a3d7682"
-          (reference "F4") (unit 1)
-        )
-      )
-    )
-  )
   (symbol (lib_id "Regulator_Linear:L78L33_SOT89") (at 101.6 224.79 0) (unit 1)
     (in_bom yes) (on_board yes) (dnp no) (fields_autoplaced)
@@
         (path "/1e139717-fcd1-4008-a6ea-4c993845e928/bcabd54f-a555-4409-9a4f-89c20a3d7682"
           (reference "#PWR04") (unit 1)
-        )
-      )
-    )
-  )
-  (symbol (lib_id "Device:Polyfuse") (at 226.06 142.24 90) (unit 1)
-    (in_bom yes) (on_board yes) (dnp no) (fields_autoplaced)
-    (property "Reference" "F3" (at 226.06 137.16 90)
-      (effects (font (size 1.27 1.27)))
-    )
-    (property "Value" "JK30-200" (at 226.06 139.7 90)
-      (effects (font (size 1.27 1.27)))
-    )
-    (property "Footprint" "Capacitor_THT:C_Disc_D11.0mm_W5.0mm_P5.00mm" (at 231.14 140.97 0)
-      (effects (font (size 1.27 1.27)) (justify left) hide)
-    )
-    (property "Datasheet" "~" (at 226.06 142.24 0)
-      (effects (font (size 1.27 1.27)) hide)
-    )
-    (pin "1")
-    (pin "2")
-    (instances
-      (project "supply"
-        (path "/1e139717-fcd1-4008-a6ea-4c993845e928/bcabd54f-a555-4409-9a4f-89c20a3d7682"
-          (reference "F3") (unit 1)
         )
       )
@@
         )
       )
+    )
+  )
+  (symbol (lib_id "Device:Fuse") (at 152.4 142.24 90) (unit 1)
+    (in_bom yes) (on_board yes) (dnp no) (fields_autoplaced)
+    (property "Reference" "F2" (at 152.4 137.16 90)
+      (effects (font (size 1.27 1.27)))
+    )
+    (property "Value" "5A" (at 152.4 139.7 90)
+      (effects (font (size 1.27 1.27)))
+    )
+    (property "Footprint" "Connector_Wire:SolderWire-0.75sqmm_1x02_P4.8mm_D1.25mm_OD2.3mm" (at 152.4 144.018 90)
+      (effects (font (size 1.27 1.27)) hide)
+    )
+    (property "Datasheet" "~" (at 152.4 142.24 0)
+      (effects (font (size 1.27 1.27)) hide)
+    )
+    (pin "1")
+    (pin "2")
+    (instances
+      (project "supply"
+        (path "/1e139717-fcd1-4008-a6ea-4c993845e928/bcabd54f-a555-4409-9a4f-89c20a3d7682"
+          (reference "F2") (unit 1)
+        )
+      )

Commit message: Board prepared to order
Parts:
- C20: value 0.1 uF -> 100 nF
Changed lines of the file:
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@@
       (effects (font (size 1.27 1.27)) (justify right))
     )
-    (property "Value" "0.1 uF" (at 116.84 231.14 0)
+    (property "Value" "100 nF" (at 116.84 231.14 0)
       (effects (font (size 1.27 1.27)) (justify right))
     )

Commit message: One board settings changed from 4-layers to 2-layers to reduce it's price
Parts:
- added R18: 1K2, Resistor_SMD:R_0805_2012Metric, symbol Device:R
- D14, D17, D9: value BL-L109EGW -> red/green, common cathode, F3
- renumbered R20 to R21, R21 to R22, R22 to R23, R23 to R24, R24 to R25, R25 to R26, R26 to R27, R27 to R28, R28 to R29, R29 to R30, R30 to R31, R31 to R32, R32 to R33, R33 to R34, R34 to R35, R35 to R36, R36 to R37, R37 to R38, R38 to R39, R39 to R40, R40 to R41, R42 to R43, R43 to R44, R44 to R45
Connections:
- net FEEDBACK: now also R18.2
- net at R18.1, U2.1: now also R18.1
Other:
- moved on the sheet: R18

Commit message: UV board size changed to 100x100 to reduce production price
Parts:
- renumbered C12 to C1, C21 to C10, C22 to C11, C23 to C12, C24 to C13, C25 to C14, C26 to C15, C27 to C16, C28 to C17, C10 to C18, C30 to C19, C13 to C2, C31 to C20, C14 to C3, C15 to C4, C16 to C5, C17 to C6, C18 to C7, C19 to C8, C20 to C9, CLR3 to CLR1, D16 to D10, D17 to D11, D1 to D12, D8 to D2, D9 to D3, D10 to D4, D11 to D5, D12 to D6, D13 to D7, D14 to D8, D15 to D9, F2 to F1, F3 to F2, F4 to F3, JP3 to JP1, JP4 to JP2, JP5 to JP3, L2 to L1, Q3 to Q1, QP1 to Q2, QP1 to Q3, R18 to R1, R28 to R10, R29 to R11, R30 to R12, R31 to R13, R32 to R14, R33 to R15, R34 to R16, R35 to R17, R36 to R18, R37 to R19, R18 to R2, R38 to R20, R39 to R21, R40 to R22, R41 to R23, R14 to R24, R43 to R25, R44 to R26, R45 to R27, R21 to R3, R22 to R4, R23 to R5, R24 to R6, R25 to R7, R26 to R8, R27 to R9, TR3 to TR1, U6 to U1, U15 to U10, U16 to U11, U8 to U3, U9 to U4, U10 to U5, U11 to U6, U12 to U7, U13 to U8, U14 to U9
