File: schematics/supply/output_5v_usb.kicad_sch (KiCad schematic)
At the start: 93 parts, among them J2 USB_A, Q1 40N06, Q2 STP13NK60Z, Q3 STP13NK60Z, U1 INA3221, U10 LM158DR, U11 LM1085-3.3, U2 EL817, U3 MC34063AD, U4 L78L33ACUTR, U5 IR2153S, U6 LM158DR, U7 IP2163, U8 LM158DR, U9 TL432DBZ

Commit message: supply board - power controllers changed; PWM logic changed
Parts:
- removed C10: 1 uF, Capacitor_SMD:C_0603_1608Metric, symbol Device:C
- removed C18: 10 nF, Capacitor_SMD:C_0603_1608Metric, symbol Device:C
- removed C6: 470 pF, Capacitor_SMD:C_0603_1608Metric, symbol Device:C
- removed JP1: SolderJumper_2_Open, Library:SolderedJumper-2P-2mm, symbol Jumper:SolderJumper_2_Open
- removed JP2, JP3: SolderJumper_2_Open, Jumper:SolderJumper-2_P1.3mm_Open_TrianglePad1.0x1.5mm, symbol Jumper:SolderJumper_2_Open
- removed Q1: 40N06, Package_TO_SOT_SMD:TO-252-2, symbol Device:Q_NMOS_GDS
- removed R10, R9: 10, Resistor_SMD:R_0805_2012Metric, symbol Device:R
- removed R2: NOT INSTALLED, Resistor_SMD:R_0805_2012Metric, symbol Device:R
- removed R64, R65, R66: 0.07, Resistor_SMD:R_2512_6332Metric, symbol Device:R
- removed U3: MC34063AD, Package_SO:SOP-8_3.9x4.9mm_P1.27mm, symbol Regulator_Switching:MC34063AD
- removed U5: IR2153S, Package_SO:SOP-8_3.76x4.96mm_P1.27mm, symbol Driver_FET:IR2153
- added C13: 1 uF, Capacitor_SMD:C_0603_1608Metric, symbol Device:C
- added C18, C23, C26: 1000 uF@16V, Capacitor_THT:CP_Radial_D10.0mm_P5.00mm, symbol Device:C_Polarized
- added C19, C25: 22 uF, Capacitor_SMD:C_1210_3225Metric, symbol Device:C
- added C5: 2 nF, Capacitor_SMD:C_0603_1608Metric, symbol Device:C
- added C7: 100 nF, Capacitor_SMD:C_0603_1608Metric, symbol Device:C
- added L3: 22 uH@0650, Inductor_SMD:L_Chilisin_BMRB00060650, symbol Device:L
- added NT1, NT2: NetTie_2, NetTie:NetTie-2_SMD_Pad2.0mm, symbol Device:NetTie_2
- added R19: 100, Resistor_SMD:R_0805_2012Metric, symbol Device:R
- added R3, R4: 10K, Resistor_SMD:R_0805_2012Metric, symbol Device:R
- added R7: 22, Resistor_SMD:R_0805_2012Metric, symbol Device:R
- added U2: XL6009, Package_TO_SOT_SMD:TO-263-5_TabPin3, symbol My_Library:XL6009
- added U5: UC3525, Package_SO:SOIC-16W_7.5x10.3mm_P1.27mm, symbol Regulator_Controller:UC3525
- added U8, U9: IR2117, Package_SO:SOIC-8_3.9x4.9mm_P1.27mm, symbol My_Library:IR2117
- C1: value 1 uF -> 100 nF
- C16: renamed from C3; value CK45-B3DD331KYGNA -> К73-17 0.022 uF@630V; footprint Capacitor_THT:C_Disc_D7.5mm_W5.0mm_P5.00mm -> Capacitor_THT:C_Rect_L13.0mm_W6.0mm_P10.00mm_FKS3_FKP3_MKS4
- C17: renamed from C5; value CK45-B3DD331KYGNA -> К73-17 0.022 uF@630V; footprint Capacitor_THT:C_Disc_D7.5mm_W5.0mm_P5.00mm -> Capacitor_THT:C_Rect_L13.0mm_W6.0mm_P10.00mm_FKS3_FKP3_MKS4
- C2: value 300 pF -> 22 uF; footprint Capacitor_SMD:C_0603_1608Metric -> Capacitor_SMD:C_1210_3225Metric
- R1: value 120 -> 220
- R15: renamed from R4; value 5K1@2W -> 100@2W
- R6: value 51 -> 5K
- renumbered C13 to C10, C12 to C14, C14 to C15, C15 to C20, C16 to C21, C17 to C22, C19 to C24, C20 to C27, C7 to C3, C8 to C4, C9 to C6, C4 to C8, C11 to C9, D2 to D1, D6 to D11, D3 to D2, D5 to D4, D7 to D5, D8 to D6, D9 to D7, D4 to D8, D11 to D9, Q2 to Q1, Q3 to Q2, R11 to R10, R12 to R11, R13 to R12, R14 to R13, R15 to R14, R18 to R16, R21 to R17, R22 to R18, R3 to R2, R16 to R20, R17 to R21, R23 to R22, R19 to R23, R20 to R24, R24 to R28, R7 to R8, R8 to R9, U8 to U10, U10 to U11, U9 to U12, U11 to U13, U2 to U3
Connections:
- net USB_3_+5V is gone; now on net USB_2_3_+5V: F3.1
- net +5V_OUT: now also C23.1, L3.1, NT1.1, NT2.1, R19.1; no longer F1.1, R20.1
- net GND: now also C18.2, C19.1, C23.2, C25.1, C26.2, U2.1 (GND); no longer C1.1, R6.2
- net GNDPWR: now also C1.2, R5.2, R6.2, C5.2, C7.2, R4.2, U5.10 (SD), U5.12 (GND), U8.3 (GND), U9.3 (GND), U9.6 (VS); no longer U3.3
- net RC_SNABBER_MIDDLEPOINT: now also C13.2, U8.6 (VS)
- net USB_1_+5V: now also C2.2, L1.2, NT1.2, U2.2 (EN), U2.4 (VIN); no longer C1.2
- net V_STANDBY: now also U5.13 (VC), U5.15 (VIN), U8.1 (VCC), U9.1 (VCC), U9.8 (VB)
- net DCDC_5V_VREF: now reaches U3.4
- net DCDC_5V_VREF: now also C1.1, R3.1, U5.16 (REF); no longer R5.1
- net at D16.1 (K): now also C13.1, U8.8 (VB)
- net at Q2.1 (G): now also U9.7 (OUT)
- net at D1.2 (A): now also L1.1, U2.3 (SW); no longer L1.2
- net at R6.1: now also U5.6 (RT)
- net at Q1.1 (G): now also U8.7 (OUT)
- net at C4.2, R8.2, R9.1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: now also U2.5 (FB)
- net at D8.2 (K), L2.1: now also C18.1, C19.2
- net USB_2_+5V renamed USB_2_3_+5V
- net USB_2_3_+5V: now also NT2.2
- new net: C5.1, R7.1, U5.5 (CT)
- new net: U5.11 (OUTA), U8.2 (IN)
- new net: U5.14 (OUTB), U9.2 (IN)
- new net: R7.2, U5.7 (DISCH)
- new net: C7.1, U5.8 (SS)
- new net: C25.2, C26.1, F1.1, L3.2
- new net: R19.2, R20.1
- new net DCDC_2V5_VREF: R3.2, R4.1, U5.2 (NI)
- new net DCDC_FEEDBACK: R5.1, U3.3, U5.1 (INV)
- no-connect marks 6 -> 9
Other:
- note removed: "100 KHz"
- note removed: "80 KHz"
- note removed: "TEST REQUIRED"
- note removed: "Use one of tbem"
- moved on the sheet: C10, C14, C15, C16, C17, C20, C21, C22, C24, C27, C3, C4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

Commit message: re-design supply board
Parts:
- removed D10, D11: SMCJ5.0A, Diode_SMD:D_SMC, symbol Diode:ESD9B3.3ST5G
- removed D4: SMAJ26A, Diode_SMD:D_SMA, symbol Diode:ESD9B3.3ST5G
- added D10, D11: SMCJ5.0A, Diode_SMD:D_SMC, symbol Diode:Z3SMCxxx
- added D4: SMAJ26A, Diode_SMD:D_SMA, symbol Diode:SMAJ26A
- added TP1: 5V_A, TestPoint:TestPoint_Pad_1.0x1.0mm, symbol Connector:TestPoint
- added TP2: 5V_B, TestPoint:TestPoint_Pad_1.0x1.0mm, symbol Connector:TestPoint
- U10, U11, U6: footprint Package_SO:SOP-8_5.28x5.23mm_P1.27mm -> Package_SO:SOP-8_3.76x4.96mm_P1.27mm
- renumbered C13 to C11, C14 to C12, C15 to C13, C16 to C14, C17 to C15, C18 to C16, C19 to C17, C20 to C18, C21 to C19, C22 to C20, C23 to C21, C24 to C22, C25 to C23, C26 to C24, C27 to C25
Connections:
- net +5V_OUT: now also D10.1 (K)
- net +5V_VSYS: now also D11.1 (K)
- net GND: now also D10.2 (A), D11.2 (A), D4.2 (A2)
- net VBUS_1: now also D4.1 (A1)
- net at U5.11 (OUTA), U8.2 (IN): now also TP1.1
- net at U5.14 (OUTB), U9.2 (IN): now also TP2.1

Commit message: Continue project
Parts:
- C5: value 2 nF -> 2.2 nF
- C8: value 1 uF -> 10 uF
- R15: value 100@2W -> 450@2W
- R19: value 100 -> 150
- R6: value 5K -> 2K2
- U1: footprint Package_DFN_QFN:Texas_RGV_S-PVQFN-N16_EP2.1x2.1mm -> Package_DFN_QFN:Texas_RGV0016A_VQFN-16-1EP_4x4mm_P0.65mm_EP2.1x2.1mm
- renumbered D16 to D3, RV1 to RV2, TP6 to TP3
Other:
- moved on the sheet: R6
