File: schematics/supply/control.kicad_sch (KiCad schematic)
At the start: 102 parts, among them J10 Conn_01x04_Pin, J11 Conn_01x04_Pin, J12 Conn_01x04_Pin, J13 Conn_01x04_Pin, J14 USBASP, J15 USBASP, J16 JST XH B3B, J17 Conn_01x06_Pin, J18 Conn_01x03_Pin, J19 Conn_01x06_Pin, M1 Fan, Q10 IRLML5203, Q3 IRLML0030, Q4 IRLML0030, Q6 IRLML0030, SW1 EC11W****, SW3 SW_Push, U14 ATmega328-A, U15 ATtiny1616-M, U16 Display_1.18inch_st7535, U17 AD9833xRM, U18 MCP4726A0T-E/CH, U19 MAX961, U20 LM158DR, U21 FAN3100, X1 HC-49U, 16MHz, X2 25 MHz

Commit message: debugging DCDC converters... Standby supply works fine (noise level = 1,7%). At now Starting to debug PFC module
Parts:
- added C60: 1 uF, Capacitor_SMD:C_0603_1608Metric, symbol Device:C
- added C82: 4.7 uF, Capacitor_SMD:C_0603_1608Metric, symbol Device:C
- added D20: BAV21WS, Diode_SMD:D_SOD-323F, symbol Device:D
- added R79: 510, Resistor_SMD:R_0805_2012Metric, symbol Device:R
- added TP25: REF_2V5, TestPoint:TestPoint_Pad_1.0x1.0mm, symbol Connector:TestPoint
- added U28: TL431DBZ, Package_TO_SOT_SMD:SOT-23, symbol Reference_Voltage:TL431DBZ
- renumbered C26 to C32, C27 to C33, C31 to C37, C32 to C38, C33 to C39, C34 to C40, C67 to C44, C68 to C45, C38 to C46, C66 to C47, C40 to C49, C69 to C50, C41 to C51, C45 to C55, C49 to C59, D13 to D14, D14 to D15, D15 to D16, D16 to D17, D17 to D18, D18 to D19, D19 to D21, D20 to D22, R29 to R32, R30 to R33, R31 to R34, R32 to R35, R33 to R36, R34 to R37, R35 to R38, R36 to R39, R38 to R42, R39 to R43, R43 to R47, R44 to R48, R45 to R49, R46 to R50, R47 to R51, TP7 to TP10, TP8 to TP11, TP9 to TP12, TP10 to TP13, TP11 to TP14, TP12 to TP15, TP13 to TP16, TP14 to TP17, TP15 to TP18, TP16 to TP19, TP4 to TP7, TP5 to TP8, TP6 to TP9, U14 to U13, U15 to U14, U16 to U15, U17 to U16, U18 to U17, U19 to U18, U20 to U19, U21 to U20
Connections:
- net +5V_VSYS: now also D20.1 (K), R79.2
- net GND: now also C60.1, C82.2, U28.3 (A)
- net IS_ONOFF_BUTTON_PRESSED: now also C60.2
- net ATTINY_VREF_2V5: now reaches U14.7 (PA6)
- net ATTINY_VREF_2V5: now also C82.1, R79.1, TP25.1, U28.1 (K), U28.2 (REF)
- net at M1.2 (-), Q6.3 (D): now also D20.2 (A)
- no-connect marks 16 -> 15
Other:
- moved on the sheet: SW3

Commit message: Board#1 schematics rewrited
Parts:
- removed C33: 100 nF, Capacitor_SMD:C_0603_1608Metric, symbol Device:C
- removed C40: 220 nF, Capacitor_SMD:C_0603_1608Metric, symbol Device:C
- removed C59, C60: 1 uF, Capacitor_SMD:C_0603_1608Metric, symbol Device:C
- removed C82: 4.7 uF, Capacitor_SMD:C_0603_1608Metric, symbol Device:C
- removed D14: GNL-3012ED, Connector_JST:JST_XH_B2B-XH-A_1x02_P2.50mm_Vertical, symbol Device:LED
- removed D15: GNL-3012GD, Connector_JST:JST_XH_B2B-XH-A_1x02_P2.50mm_Vertical, symbol Device:LED
- removed D21, D22: BAV21WS, Diode_SMD:D_SOD-323F, symbol Device:D
- removed J15: USBASP, Library:DC3-2x05_p2.54, symbol Connector_Generic:Conn_02x05_Odd_Even
- removed J16: JST XH B3B, Connector_JST:JST_XH_B3B-XH-A_1x03_P2.50mm_Vertical, symbol Connector:Conn_01x03_Socket
- removed J18: Conn_01x03_Pin, symbol Connector:Conn_01x03_Pin
- removed Q3, Q4: IRLML0030, Package_TO_SOT_SMD:SOT-23, symbol Transistor_FET:IRLML0030
- removed R33, R34, R38, R49, R50, R51: 10K, Resistor_SMD:R_0805_2012Metric, symbol Device:R
- removed R36, R39: 220, Resistor_SMD:R_0805_2012Metric, symbol Device:R
- removed R79: 510, Resistor_SMD:R_0805_2012Metric, symbol Device:R
- removed SW3: SW_Push, Connector_JST:JST_XH_B2B-XH-A_1x02_P2.50mm_Vertical, symbol Switch:SW_Push
- removed TP16: BTN_FB, TestPoint:TestPoint_Pad_1.0x1.0mm, symbol Connector:TestPoint
- removed TP17: IC_FB, TestPoint:TestPoint_Pad_1.0x1.0mm, symbol Connector:TestPoint
- removed TP19: PW_FB, TestPoint:TestPoint_Pad_1.0x1.0mm, symbol Connector:TestPoint
- removed TP25: REF_2V5, TestPoint:TestPoint_Pad_1.0x1.0mm, symbol Connector:TestPoint
- removed TP7: PW_CS, TestPoint:TestPoint_Pad_1.0x1.0mm, symbol Connector:TestPoint
- removed TP8: PW_VS, TestPoint:TestPoint_Pad_1.0x1.0mm, symbol Connector:TestPoint
- removed TP9: PW_SHDN#, TestPoint:TestPoint_Pad_1.0x1.0mm, symbol Connector:TestPoint
- removed U14: ATtiny1616-M, Package_DFN_QFN:VQFN-20-1EP_3x3mm_P0.4mm_EP1.7x1.7mm, symbol MCU_Microchip_ATtiny:ATtiny1616-M
- removed U20: FAN3100, Package_TO_SOT_SMD:SOT-23-5, symbol My_Library:FAN3100
- removed U28: TL431DBZ, Package_TO_SOT_SMD:SOT-23, symbol Reference_Voltage:TL431DBZ
- added C20: 1000 uF@16V, Capacitor_THT:CP_Radial_D10.0mm_P5.00mm, symbol Device:C_Polarized
- added C22: 22 uF, Capacitor_SMD:C_1210_3225Metric, symbol Device:C
- added F4: Fuse, Library:FuseHolder1808, symbol Device:Fuse
- renumbered C32 to C21, C37 to C26, C38 to C27, C39 to C28, C44 to C32, C45 to C33, C46 to C34, C47 to C35, C49 to C37, C50 to C38, C51 to C39, C55 to C43, D18 to D10, D19 to D11, D20 to D12, D16 to D8, D17 to D9, J13 to J10, J14 to J11, J17 to J12, J19 to J13, J10 to J7, J11 to J8, J12 to J9, Q6 to Q3, R32 to R20, R35 to R21, R37 to R22, R42 to R25, R43 to R26, R47 to R30, R48 to R31, RV3 to RV1, RV4 to RV2, TP10 to TP1, TP11 to TP2, TP12 to TP3, TP13 to TP4, TP14 to TP5, TP15 to TP6, TP18 to TP7, U13 to U11, U15 to U12, U16 to U13, U17 to U14, U18 to U15, U19 to U16
Connections:
- net SIGNAL_OUT: now also D11.1 (K), R30.2, U15.6 (Q)
- net +5V_VSYS renamed VSYS
- net VSYS: now also C20.1, C22.2, F4.2
- net GND renamed VSYS_GND
- net VSYS_GND: now also C20.2, C22.1
- net IS_ONOFF_BUTTON_PRESSED: no longer names the net of U11.12 (PB0)
- new net VSYS_VCC: F4.1
- no-connect marks 15 -> 6
Other:
- note removed: "ATTiny program port"
- note removed: "I2C address: 0x33"
- note removed: "vdd cap"
- moved on the sheet: C21, C26, C27, C28, C35, C36, C37, C43, J10, J11, J7, J8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

Commit message: added some protection logic
Parts:
- renumbered C38 to C40, C39 to C43, C43 to C45, R31 to R27, R30 to R31, U16 to U15, U15 to U16
Connections:
- net SIGNAL_GEN_SHTDN: now also U11.12 (PB0); no longer U11.30 (PD0)
- net RXD: now reaches J11.4 (Pin_4)
- net RXD: now also U11.30 (PD0)
- no-connect marks 6 -> 4
Other:
- moved on the sheet: C21, C26, C27, C28, C32, C33, C34, C35, C36, C37, C40, C43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

Commit message: first board routed
Parts:
- removed C20: 1000 uF@16V, Capacitor_THT:CP_Radial_D10.0mm_P5.00mm, symbol Device:C_Polarized
- removed C22: 22 uF, Capacitor_SMD:C_1210_3225Metric, symbol Device:C
- removed F4: Fuse, Library:FuseHolder1808, symbol Device:Fuse
- added C54: 1 uF, Capacitor_SMD:C_0603_1608Metric, symbol Device:C
Connections:
- net VSYS is gone; now on net VSYS_VCC: C21.1, C32.1, C33.1, C34.1, C35.1, C36.2, C37.1, C45.1, D12.1 (K), J11.2 (Pin_2), JP1.3 (B), M1.1 (+), Q10.2 (S), R20.2, R21.2, R22.2, R32.2, R32.2, R32.2, RV1.1, RV2.1, TH1.1, TH2.1, U11.18 (AVCC), U11.20 (AREF), U11.4 (VCC), U11.6 (VCC), U13.2 (VDD), U14.3 (VDD), U14.6 (VREF), U15.8 (V+), U16.8 (VCC), X2.4 (Vcc)
- net VSYS_GND: now also C54.2
- net VSYS_VCC: now also C54.1

Commit message: some changes in board routing
Parts:
- renumbered C21 to C23, C26 to C27, C27 to C28, C28 to C29, C32 to C33, C33 to C34, C34 to C35, C35 to C36, C37 to C38, C40 to C41, C43 to C44, C45 to C46, C54 to C48, J7 to J10, J8 to J11, J9 to J12, J10 to J13, J11 to J14, J12 to J15, J13 to J16, R20 to R22, R21 to R23, R22 to R24, R25 to R27, R26 to R28, R27 to R29, R31 to R33
