File: schematics/supply-uv/supply-uv.kicad_pcb (KiCad board)
At the start: 2 copper layers, 120 x 200 mm, 284 parts, among them J1 VSYS connector to Board#2, J2 power +5V connector to board#2, J3 +5V_PWR (with fuse), J4 PWR_OUT (with fuse), J5 CW2B-10A-T, J6 USBASP, J7 JST XH B3B, K1 SRD-12VDC-SL-C, Q1 5N65F, Q10 STP13NK60Z, Q11 STP13NK60Z, Q12 IRLML0030, Q13 IRLML0030, Q14 IRLML0030, Q2 IRLML5203, Q3 IRLML5203, Q4 IRLML5203, Q5 STP13NK60Z, Q6 STP13NK60Z, Q7 IRLML0030, Q8 IRLML5203, Q9 IRLML0030, SW1 SW_Push, U1 ISO1540, U10 TL331, U11 EL817, U12 UC3525, U13 IRS21867S, U14 TL432DBZ, U15 EL817, U16 UC3525, U17 OP213ESZ, U18 IRS21867S, U19 EL817, U2 R7731, U20 INA169, U21 TL431DBZ, U22 ATtiny1616-M, U3 EL817, U4 EL817, U5 L7805ABV, U6 L7805ABV, U7 TL431DBZ, U8 EL817, U9 TL432DBZ, Y1 B32022A3223M000

Commit message: First board routing completed. I will review it few days later and maybe optimize something, but base worki done
Parts:
- removed the TP18 at (-72.9, 221.3)
- removed the TP19 at (-72.9, 223.8)
- removed the TP29 at (121.1, 195.0)
- removed the TP30 at (121.1, 197.5)
- added C38: 100 nF, Capacitor_SMD:C_0603_1608Metric, F.Cu at (74.9, 127.5)
- added C59: 100 nF, Capacitor_SMD:C_0603_1608Metric, F.Cu at (108.3, 139.4)
- added JP6: Overpower mode, Connector_PinSocket_2.54mm:PinSocket_1x03_P2.54mm_Vertical, F.Cu at (71.4, 149.5)
- added JP7: Overpower mode, Connector_PinSocket_2.54mm:PinSocket_1x03_P2.54mm_Vertical, F.Cu at (135.9, 139.8)
- C31, C33, C34, C35, C37, L5, NT3, Q12, Q7, Q8, Q9, U12, U14, U17, U20: moved to B.Cu
- C46: renamed from C45; moved to B.Cu
- C48: renamed from C47; moved to B.Cu
- C49: renamed from C48; moved to B.Cu
- C50: renamed from C49; moved to B.Cu
- C54: renamed from C53; moved to B.Cu
- C55: renamed from C54; moved to B.Cu
- C58: renamed from C57; moved to B.Cu
- C63: renamed from C61; moved to B.Cu
- C69: renamed from C67; moved to B.Cu
- C70: renamed from C68; moved to B.Cu
- C71: renamed from C69; moved to B.Cu
- D14, D19: value SMBJ3.3A -> SM6T30CA; moved to B.Cu
- NT1: footprint NetTie:NetTie-2_SMD_Pad2.0mm -> NetTie:NetTie-2_SMD_Pad0.5mm
- R31: renamed from R29; moved to B.Cu
- R32: renamed from R31; moved to B.Cu
- R33: renamed from R30; moved to B.Cu
- R36: renamed from R34; moved to B.Cu
- R37: renamed from R35; moved to B.Cu
- R38: renamed from R36; moved to B.Cu
- R41: renamed from R39; moved to B.Cu
- R42: renamed from R40; moved to B.Cu
- R43: renamed from R41; moved to B.Cu
- R44: renamed from R42; moved to B.Cu
- R45: renamed from R43; moved to B.Cu
- R46: renamed from R44; moved to B.Cu
- R49: renamed from R47; moved to B.Cu
- R50: renamed from R48; moved to B.Cu
- R51: renamed from R49; moved to B.Cu
- R53: renamed from R51; moved to B.Cu
- R54: renamed from R52; moved to B.Cu
- R55: renamed from R53; moved to B.Cu
- R56: renamed from R54; moved to B.Cu
- R60: renamed from R58; moved to B.Cu
- R62: renamed from R60; moved to B.Cu
- R64: renamed from R62; moved to B.Cu
- R65: renamed from R63; moved to B.Cu
- R66: renamed from R64; moved to B.Cu
- R67: renamed from R65; moved to B.Cu
- TP10, TP9: footprint TestPoint:TestPoint_Pad_2.0x2.0mm -> TestPoint:TestPoint_Pad_1.0x1.0mm
- TP20: renamed from TP22; footprint Library:TestPoint_Plated_Hole_D1.0mm -> TestPoint:TestPoint_Pad_1.0x1.0mm
- TP26: renamed from TP28; footprint Library:TestPoint_Plated_Hole_D1.0mm -> TestPoint:TestPoint_Pad_1.0x1.0mm
- TP6: value VSYS2_VCC -> VSYS2
- moved C32 512.0 mm to (94.7, 113.5), turned to 90 degrees
- moved C36 507.7 mm to (99.5, 111.7), turned to -90 degrees
- moved R35 503.7 mm to (76.9, 130.9), turned to -90 degrees
- moved R37 503.4 mm to (81.0, 135.2)
- moved R38 503.4 mm to (81.0, 137.3), turned to 180 degrees
- moved R34 498.0 mm to (71.2, 129.7)
- moved C35 489.5 mm to (80.7, 133.3)
- moved C37 486.7 mm to (80.8, 139.3)
- moved C30 482.1 mm to (72.8, 132.4)
- moved U12 480.6 mm to (71.2, 134.1), turned to 180 degrees
- moved R36 479.2 mm to (80.1, 148.7)
- moved R33 478.2 mm to (77.9, 194.2)
- moved C33 477.0 mm to (67.3, 140.7)
- moved R32 476.5 mm to (49.1, 156.1)
- moved R31 476.5 mm to (75.4, 197.6), turned to -90 degrees
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- renumbered C38 to C39, C39 to C40, C40 to C41, C41 to C42, C42 to C43, C43 to C44, C44 to C45, C46 to C47, C50 to C51, C51 to C52, C52 to C53, C55 to C56, C56 to C57, C58 to C60, C59 to C61, C60 to C62, C62 to C64, C63 to C65, C64 to C66, C65 to C67, C66 to C68, C70 to C72, C71 to C73, C72 to C74, C73 to C75, JP4 to JP1, JP5 to JP2, JP1 to JP3, JP2 to JP4, JP3 to JP5, RP1 to R26, RP2 to R27, R26 to R28, R27 to R29, R28 to R30, R32 to R34, R33 to R35, R37 to R39, R38 to R40, R45 to R47, R46 to R48, R50 to R52, R55 to R57, R56 to R58, R57 to R59, R59 to R61, R61 to R63, R66 to R68, R67 to R69, R68 to R70, R69 to R71, R70 to R72, R71 to R73, R72 to R74, R73 to R75, R74 to R76, TP20 to TP18, TP21 to TP19, TP23 to TP21, TP24 to TP22, TP25 to TP23, TP26 to TP24, TP27 to TP25, TP31 to TP27, TP32 to TP28, TP33 to TP29, TP34 to TP30, TP35 to TP31, TP36 to TP32, TP37 to TP33, TP38 to TP34
Connections:
- C31 pad 1: /5V_PWR Sheet/DCDC_SHUTDOWN -> Net-(D14-A2)
- C31 pad 2: /5V_PWR Sheet/STB_GND -> /5V_PWR Sheet/HV_GND
- C54 pad 1: Net-(D19-A1) -> Net-(D19-A2)
- C54 pad 2: /5V_PWR Sheet/STB_GND -> /5V_PWR Sheet/HV_GND
- C63 pad 1: /pwrout Sheet/DCDC_5V_VREF -> /pwrout Sheet/STB_VCC
- C63 pad 2: /5V_PWR Sheet/STB_GND -> /5V_PWR Sheet/HV_GND
- D14 pad 1: /5V_PWR Sheet/DCDC_SHUTDOWN -> /5V_PWR Sheet/HV_GND
- D14 pad 2: /5V_PWR Sheet/STB_GND -> Net-(D14-A2)
- D19 pad 1: Net-(D19-A1) -> /5V_PWR Sheet/HV_GND
- D19 pad 2: /5V_PWR Sheet/STB_GND -> Net-(D19-A2)
- Q8 pad 3: Net-(Q8-D) -> Net-(JP7-B)
- R32 pad 2: /5V_PWR Sheet/DCDC_SHUTDOWN -> Net-(D14-A2)
- R46 pad 2: Net-(D19-A1) -> Net-(D19-A2)
- R54 pad 1: /5V_PWR Sheet/STB_GND -> /5V_PWR Sheet/HV_GND
- TR1 pad 2: /VSYS_PWR_GND -> /VSYS_GND
- TR1 pad 4: Net-(D7-A) -> Net-(D6-A)
- TR1 pad 6: /VSYS_GND -> /VSYS_PWR_GND
- TR1 pad 8: Net-(D6-A) -> Net-(D7-A)
- U15 pad 4: Net-(Q8-D) -> Net-(JP7-C)
- U17 pad 3: Net-(D19-A1) -> Net-(D19-A2)
- U17 pad 4: /5V_PWR Sheet/STB_GND -> /5V_PWR Sheet/HV_GND
- U17 pad 8: /pwrout Sheet/DCDC_5V_VREF -> /pwrout Sheet/STB_VCC
Routing:
- net /5V_PWR Sheet/HV_GND: track 200.7 -> 648.0 mm
- net /+5V_PWR_GND: track 0.00 -> 408.8 mm
- net /5V_PWR Sheet/STB_GND: track 156.8 -> 454.0 mm, vias 1 -> 7
- net /pwrout Sheet/PWR_GND: track 0.00 -> 260.3 mm, vias 0 -> 1
- net /pwrout Sheet/HV_VCC_FUSE: track 0.00 -> 174.9 mm, vias 0 -> 9
- net /+5V_PWR_VCC: track 0.00 -> 158.9 mm, vias 0 -> 9
- net Net-(D21-A-Pad3): track 0.00 -> 147.8 mm
- net /5V_PWR Sheet/STB_VCC: track 0.00 -> 117.8 mm, vias 0 -> 1
- net Net-(Q10-S): track 0.00 -> 111.1 mm, vias 0 -> 1
- net /VSYS_PWR_GND: track 274.3 -> 385.2 mm
- net /pwrout Sheet/STB_VCC: track 0.00 -> 104.9 mm, vias 0 -> 5
- net Net-(D16-A-Pad1): track 0.00 -> 90.2 mm
- net Net-(D16-K): track 0.00 -> 78.0 mm, vias 0 -> 9
- net Net-(Q5-S): track 0.00 -> 76.4 mm
- net Net-(D21-A-Pad1): track 0.00 -> 75.9 mm
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Other:
- board size 120 x 200 mm -> 150 x 200 mm
- board text added: "150,0000 mm x 200,0000 mm"
- board text added: "Supply-hv v2.0"
- board text removed: "100,0000 mm x 100,0000 mm"
