File: schematics/supply-uv/5v_pwr.kicad_sch (KiCad schematic)
At the start: 62 parts, among them Q5 STP13NK60Z, Q6 STP13NK60Z, U11 EL817, U12 UC3525, U13 IRS21867S, U14 TL432DBZ

Commit message: Boards prepared to order
Parts:
- renumbered C30 to C31, C31 to C32, C32 to C33, C33 to C34, C34 to C35, C35 to C36, C36 to C37, C37 to C38, C38 to C39, C39 to C40, C40 to C41, C41 to C42, C42 to C43, C43 to C45, C45 to C46, C46 to C47, C47 to C48, C48 to C49, C49 to C50, C50 to C51, TP10 to TP12, TP11 to TP13, TP12 to TP14, TP13 to TP15, TP14 to TP16, TP15 to TP17, TP16 to TP18, TP17 to TP19
Changed lines of the file:
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@@
 		(on_board yes)
 		(dnp no)
-		(property "Reference" "C48"
+		(property "Reference" "C49"
 			(at 394.208 111.76 0)
 			(effects
@@
 			(project "supply-uv"
 				(path "/ef40850c-d0bf-4cba-961b-9aba418f8e73/c057ed5d-9c60-40b5-98c1-144531018637"
-					(reference "C48")
+					(reference "C49")
 					(unit 1)
 				)
@@
 		(dnp no)
 		(fields_autoplaced yes)
-		(property "Reference" "TP16"
+		(property "Reference" "TP18"
 			(at 224.79 95.7579 0)
 			(effects
@@
 			(project "supply-uv"
 				(path "/ef40850c-d0bf-4cba-961b-9aba418f8e73/c057ed5d-9c60-40b5-98c1-144531018637"
-					(reference "TP16")
+					(reference "TP18")
 					(unit 1)
 				)
@@
 		(on_board yes)
 		(dnp no)
-		(property "Reference" "C43"
+		(property "Reference" "C45"
 			(at 288.29 51.816 0)
 			(effects
@@
 			(project "supply-uv"
 				(path "/ef40850c-d0bf-4cba-961b-9aba418f8e73/c057ed5d-9c60-40b5-98c1-144531018637"
-					(reference "C43")
+					(reference "C45")
 					(unit 1)
 				)
@@
 		(on_board yes)
 		(dnp no)
-		(property "Reference" "C35"
+		(property "Reference" "C36"
 			(at 118.364 111.76 0)
 			(effects
@@
 			(project "supply-uv"
 				(path "/ef40850c-d0bf-4cba-961b-9aba418f8e73/c057ed5d-9c60-40b5-98c1-144531018637"
-					(reference "C35")
+					(reference "C36")
 					(unit 1)
 				)
@@
 		(dnp no)
 		(fields_autoplaced yes)
-		(property "Reference" "TP14"
+		(property "Reference" "TP16"
 			(at 189.23 151.6379 0)
 			(effects
@@
 			(project "supply-uv"
 				(path "/ef40850c-d0bf-4cba-961b-9aba418f8e73/c057ed5d-9c60-40b5-98c1-144531018637"
-					(reference "TP14")
+					(reference "TP16")
 					(unit 1)
 				)
@@
 		(on_board yes)
 		(dnp no)
-		(property "Reference" "C39"
+		(property "Reference" "C40"
 			(at 191.77 120.65 0)
 			(effects
@@
 			(project "supply-uv"
 				(path "/ef40850c-d0bf-4cba-961b-9aba418f8e73/c057ed5d-9c60-40b5-98c1-144531018637"
-					(reference "C39")
+					(reference "C40")
 					(unit 1)
 				)
@@
 		(dnp no)
 		(fields_autoplaced yes)
-		(property "Reference" "TP12"
+		(property "Reference" "TP14"
 			(at 167.64 89.4079 0)
 			(effects
@@
 			(project "supply-uv"
 				(path "/ef40850c-d0bf-4cba-961b-9aba418f8e73/c057ed5d-9c60-40b5-98c1-144531018637"
-					(reference "TP12")
+					(reference "TP14")
 					(unit 1)
 				)
@@
 		(on_board yes)
 		(dnp no)
-		(property "Reference" "C37"
+		(property "Reference" "C38"
 			(at 133.35 111.76 0)
 			(effects
@@
 			(project "supply-uv"
 				(path "/ef40850c-d0bf-4cba-961b-9aba418f8e73/c057ed5d-9c60-40b5-98c1-144531018637"
-					(reference "C37")
+					(reference "C38")
 					(unit 1)
 				)
@@
 		(on_board yes)
 		(dnp no)
-		(property "Reference" "C33"
+		(property "Reference" "C34"
 			(at 103.632 87.63 0)
 			(effects
@@
 			(project "supply-uv"
 				(path "/ef40850c-d0bf-4cba-961b-9aba418f8e73/c057ed5d-9c60-40b5-98c1-144531018637"
-					(reference "C33")
+					(reference "C34")
 					(unit 1)
 				)
@@
 		(dnp no)
 		(fields_autoplaced yes)
-		(property "Reference" "TP10"
+		(property "Reference" "TP12"
 			(at 109.22 149.0979 0)
 			(effects
@@
 			(project "supply-uv"
 				(path "/ef40850c-d0bf-4cba-961b-9aba418f8e73/c057ed5d-9c60-40b5-98c1-144531018637"
-					(reference "TP10")
+					(reference "TP12")
 					(unit 1)
 				)
@@
 		(on_board yes)
 		(dnp no)
-		(property "Reference" "C31"
+		(property "Reference" "C32"
 			(at 59.69 129.54 0)
 			(effects
@@
 			(project "supply-uv"
 				(path "/ef40850c-d0bf-4cba-961b-9aba418f8e73/c057ed5d-9c60-40b5-98c1-144531018637"
-					(reference "C31")
+					(reference "C32")
 					(unit 1)
 				)
@@
 		(on_board yes)
 		(dnp no)
-		(property "Reference" "C32"
+		(property "Reference" "C33"
 			(at 99.822 52.832 0)
 			(effects
@@
 			(project "supply-uv"
 				(path "/ef40850c-d0bf-4cba-961b-9aba418f8e73/c057ed5d-9c60-40b5-98c1-144531018637"
-					(reference "C32")
+					(reference "C33")
 					(unit 1)
 				)
@@
 		(on_board yes)
 		(dnp no)
-		(property "Reference" "C50"
+		(property "Reference" "C51"
 			(at 407.67 111.76 0)
 			(effects
@@
 			(project "supply-uv"
 				(path "/ef40850c-d0bf-4cba-961b-9aba418f8e73/c057ed5d-9c60-40b5-98c1-144531018637"
-					(reference "C50")
+					(reference "C51")
 					(unit 1)
 				)
@@
 		(dnp no)
 		(fields_autoplaced yes)
-		(property "Reference" "TP15"
+		(property "Reference" "TP17"
 			(at 224.79 77.9779 0)
 			(effects
@@
 			(project "supply-uv"
 				(path "/ef40850c-d0bf-4cba-961b-9aba418f8e73/c057ed5d-9c60-40b5-98c1-144531018637"
-					(reference "TP15")
+					(reference "TP17")
 					(unit 1)
 				)
@@
 		(on_board yes)
 		(dnp no)
-		(property "Reference" "C34"
+		(property "Reference" "C35"
 			(at 111.76 160.02 0)
 			(effects
@@
 			(project "supply-uv"
 				(path "/ef40850c-d0bf-4cba-961b-9aba418f8e73/c057ed5d-9c60-40b5-98c1-144531018637"
-					(reference "C34")
+					(reference "C35")
 					(unit 1)
 				)
@@
 		(dnp no)
 		(fields_autoplaced yes)
-		(property "Reference" "C41"
+		(property "Reference" "C42"
 			(at 251.46 51.1809 0)
 			(effects
@@
 			(project "supply-uv"
 				(path "/ef40850c-d0bf-4cba-961b-9aba418f8e73/c057ed5d-9c60-40b5-98c1-144531018637"
-					(reference "C41")
+					(reference "C42")
 					(unit 1)
 				)
@@
 		(dnp no)
 		(fields_autoplaced yes)
-		(property "Reference" "C46"
+		(property "Reference" "C47"
 			(at 351.79 109.855 0)
 			(effects
@@
 			(project "supply-uv"
 				(path "/ef40850c-d0bf-4cba-961b-9aba418f8e73/c057ed5d-9c60-40b5-98c1-144531018637"
-					(reference "C46")
+					(reference "C47")
 					(unit 1)
 				)
@@
 		(on_board yes)
 		(dnp no)
-		(property "Reference" "C47"
+		(property "Reference" "C48"
 			(at 373.38 115.57 0)
 			(effects
@@
 			(project "supply-uv"
 				(path "/ef40850c-d0bf-4cba-961b-9aba418f8e73/c057ed5d-9c60-40b5-98c1-144531018637"
-					(reference "C47")
+					(reference "C48")
 					(unit 1)
 				)
@@
 		(on_board yes)
 		(dnp no)
-		(property "Reference" "C45"
+		(property "Reference" "C46"
 			(at 330.2 114.3 0)
 			(effects
@@
 			(project "supply-uv"
 				(path "/ef40850c-d0bf-4cba-961b-9aba418f8e73/c057ed5d-9c60-40b5-98c1-144531018637"
-					(reference "C45")
+					(reference "C46")
 					(unit 1)
 				)
@@
 		(on_board yes)
 		(dnp no)
-		(property "Reference" "C38"
+		(property "Reference" "C39"
 			(at 162.56 121.92 0)
 			(effects
@@
 			(project "supply-uv"
 				(path "/ef40850c-d0bf-4cba-961b-9aba418f8e73/c057ed5d-9c60-40b5-98c1-144531018637"
-					(reference "C38")
+					(reference "C39")
 					(unit 1)
 				)
@@
 		(dnp no)
 		(fields_autoplaced yes)
-		(property "Reference" "C36"
+		(property "Reference" "C37"
 			(at 118.11 53.3399 0)
 			(effects
@@
 			(project "supply-uv"
 				(path "/ef40850c-d0bf-4cba-961b-9aba418f8e73/c057ed5d-9c60-40b5-98c1-144531018637"
-					(reference "C36")
+					(reference "C37")
 					(unit 1)
 				)
@@
 		(dnp no)
 		(fields_autoplaced yes)
-		(property "Reference" "TP13"
+		(property "Reference" "TP15"
 			(at 189.23 142.7479 0)
 			(effects
@@
 			(project "supply-uv"
 				(path "/ef40850c-d0bf-4cba-961b-9aba418f8e73/c057ed5d-9c60-40b5-98c1-144531018637"
-					(reference "TP13")
+					(reference "TP15")
 					(unit 1)
 				)
@@
 		(on_board yes)
 		(dnp no)
-		(property "Reference" "C42"
+		(property "Reference" "C43"
 			(at 271.78 133.35 90)
 			(effects
@@
 			(project "supply-uv"
 				(path "/ef40850c-d0bf-4cba-961b-9aba418f8e73/c057ed5d-9c60-40b5-98c1-144531018637"
-					(reference "C42")
+					(reference "C43")
 					(unit 1)
 				)
@@
 		(on_board yes)
 		(dnp no)
-		(property "Reference" "C40"
+		(property "Reference" "C41"
 			(at 201.93 88.9 0)
 			(effects
@@
 			(project "supply-uv"
 				(path "/ef40850c-d0bf-4cba-961b-9aba418f8e73/c057ed5d-9c60-40b5-98c1-144531018637"
-					(reference "C40")
+					(reference "C41")
 					(unit 1)
 				)
@@
 		(on_board yes)
 		(dnp no)
-		(property "Reference" "C30"
+		(property "Reference" "C31"
 			(at 55.88 101.6 0)
 			(effects
@@
 			(project "supply-uv"
 				(path "/ef40850c-d0bf-4cba-961b-9aba418f8e73/c057ed5d-9c60-40b5-98c1-144531018637"
-					(reference "C30")
+					(reference "C31")
 					(unit 1)
 				)
@@
 		(dnp no)
 		(fields_autoplaced yes)
-		(property "Reference" "TP11"
+		(property "Reference" "TP13"
 			(at 167.64 79.2479 0)
 			(effects
@@
 			(project "supply-uv"
 				(path "/ef40850c-d0bf-4cba-961b-9aba418f8e73/c057ed5d-9c60-40b5-98c1-144531018637"
-					(reference "TP11")
+					(reference "TP13")
 					(unit 1)
 				)
@@
 		(on_board yes)
 		(dnp no)
-		(property "Reference" "C49"
+		(property "Reference" "C50"
 			(at 398.78 137.16 0)
 			(effects
@@
 			(project "supply-uv"
 				(path "/ef40850c-d0bf-4cba-961b-9aba418f8e73/c057ed5d-9c60-40b5-98c1-144531018637"
-					(reference "C49")
+					(reference "C50")
 					(unit 1)
 				)
@@
 		(dnp no)
 		(fields_autoplaced yes)
-		(property "Reference" "TP17"
+		(property "Reference" "TP19"
 			(at 266.7 86.8679 0)
 			(effects
@@
 			(project "supply-uv"
 				(path "/ef40850c-d0bf-4cba-961b-9aba418f8e73/c057ed5d-9c60-40b5-98c1-144531018637"
-					(reference "TP17")
+					(reference "TP19")
 					(unit 1)
 				)

Commit message: power board works (except power output driver, not tested yet), I ready to solder control board
Parts:
- C35, C50: now not fitted
- C41: value 1 uF -> 47 nF .... 120 nF *; Actual (none) -> 100 nF
- D14: value SM6T30CA -> SMAJ5.0CA-TR
- R32: value 220 -> 200
- R36: value 4K7 -> 1K2
Changed lines of the file:
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@@
 	(label "DCDC_SHUTDOWN"
 		(at 127 90.17 180)
-		(fields_autoplaced yes)
 		(effects
 			(font
@@
 	(label "DCDC_CURRENT_SENSE"
 		(at 240.03 107.95 0)
-		(fields_autoplaced yes)
 		(effects
 			(font
@@
 	(label "DCDC_FEEDBACK"
 		(at 114.3 156.21 0)
-		(fields_autoplaced yes)
 		(effects
 			(font
@@
 	(label "HV_VCC_FUSE"
 		(at 83.82 22.86 0)
-		(fields_autoplaced yes)
 		(effects
 			(font
@@
 	(label "HV_VCC_FUSE"
 		(at 276.86 44.45 180)
-		(fields_autoplaced yes)
 		(effects
 			(font
@@
 	(label "FEEDBACK"
 		(at 372.11 132.08 180)
-		(fields_autoplaced yes)
 		(effects
 			(font
@@
 	(label "DCDC_CURRENT_SENSE"
 		(at 276.86 62.23 180)
-		(fields_autoplaced yes)
 		(effects
 			(font
@@
 	(label "DCDC_5V_VREF"
 		(at 63.5 87.63 180)
-		(fields_autoplaced yes)
 		(effects
 			(font
@@
 	(label "DCDC_FEEDBACK"
 		(at 127 82.55 180)
-		(fields_autoplaced yes)
 		(effects
 			(font
@@
 	(label "DCDC_5V_VREF"
 		(at 86.36 151.13 0)
-		(fields_autoplaced yes)
 		(effects
 			(font
@@
 	(label "HV_VCC_FUSE"
 		(at 236.22 71.12 180)
-		(fields_autoplaced yes)
 		(effects
 			(font
@@
 	(label "DCDC_2V5_VREF"
 		(at 64.77 100.33 0)
-		(fields_autoplaced yes)
 		(effects
 			(font
@@
 	(label "HV_VCC_FUSE"
 		(at 251.46 140.97 180)
-		(fields_autoplaced yes)
 		(effects
 			(font
@@
 	(label "FEEDBACK"
 		(at 44.45 167.64 180)
-		(fields_autoplaced yes)
 		(effects
 			(font
@@
 	(label "DCDC_SHUTDOWN"
 		(at 83.82 120.65 0)
-		(fields_autoplaced yes)
 		(effects
 			(font
@@
 	(label "DCDC_5V_VREF"
 		(at 62.23 43.18 180)
-		(fields_autoplaced yes)
 		(effects
 			(font
@@
 	(label "DCDC_5V_VREF"
 		(at 127 87.63 180)
-		(fields_autoplaced yes)
 		(effects
 			(font
@@
 	(label "DCDC_2V5_VREF"
 		(at 127 80.01 180)
-		(fields_autoplaced yes)
 		(effects
 			(font
@@
 	(label "DCDC_CURRENT_SENSE"
 		(at 36.83 125.73 180)
-		(fields_autoplaced yes)
 		(effects
 			(font
@@
 	(label "DCDC_5V_VREF"
 		(at 48.26 96.52 180)
-		(fields_autoplaced yes)
 		(effects
 			(font
@@
 	(label "HV_VCC_FUSE"
 		(at 241.3 44.45 180)
-		(fields_autoplaced yes)
 		(effects
 			(font
@@
 		(shape input)
 		(at 391.16 121.92 180)
-		(fields_autoplaced yes)
 		(effects
 			(font
@@
 		(shape input)
 		(at 63.5 111.76 180)
-		(fields_autoplaced yes)
 		(effects
 			(font
@@
 		(shape input)
 		(at 184.15 128.27 180)
-		(fields_autoplaced yes)
 		(effects
 			(font
@@
 		(shape input)
 		(at 181.61 147.32 180)
-		(fields_autoplaced yes)
 		(effects
 			(font
@@
 		(shape input)
 		(at 144.78 67.31 90)
-		(fields_autoplaced yes)
 		(effects
 			(font
@@
 		(shape input)
 		(at 96.52 95.25 180)
-		(fields_autoplaced yes)
 		(effects
 			(font
@@
 		(shape input)
 		(at 431.8 125.73 270)
-		(fields_autoplaced yes)
 		(effects
 			(font
@@
 		(shape input)
 		(at 467.36 130.81 270)
-		(fields_autoplaced yes)
 		(effects
 			(font
@@
 		(shape input)
 		(at 184.15 115.57 180)
-		(fields_autoplaced yes)
 		(effects
 			(font
@@
 		(shape input)
 		(at 92.71 48.26 180)
-		(fields_autoplaced yes)
 		(effects
 			(font
@@
 		(shape input)
 		(at 96.52 60.96 180)
-		(fields_autoplaced yes)
 		(effects
 			(font
@@
 		(shape input)
 		(at 284.48 140.97 0)
-		(fields_autoplaced yes)
 		(effects
 			(font
@@
 		(shape input)
 		(at 72.39 115.57 180)
-		(fields_autoplaced yes)
 		(effects
 			(font
@@
 		(shape input)
 		(at 448.31 125.73 270)
-		(fields_autoplaced yes)
 		(effects
 			(font
@@
 		(shape input)
 		(at 67.31 22.86 180)
-		(fields_autoplaced yes)
 		(effects
 			(font
@@
 		(shape input)
 		(at 35.56 151.13 180)
-		(fields_autoplaced yes)
 		(effects
 			(font
@@
 		(shape input)
 		(at 143.51 113.03 270)
-		(fields_autoplaced yes)
 		(effects
 			(font
@@
 		(shape input)
 		(at 186.69 110.49 180)
-		(fields_autoplaced yes)
 		(effects
 			(font
@@
 		(shape input)
 		(at 416.56 157.48 180)
-		(fields_autoplaced yes)
 		(effects
 			(font
@@
 		(shape input)
 		(at 154.94 116.84 180)
-		(fields_autoplaced yes)
 		(effects
 			(font
@@
 		(shape input)
 		(at 347.98 118.11 270)
-		(fields_autoplaced yes)
 		(effects
 			(font
@@
 		(shape input)
 		(at 181.61 156.21 180)
-		(fields_autoplaced yes)
 		(effects
 			(font
@@
 		(shape input)
 		(at 125.73 121.92 270)
-		(fields_autoplaced yes)
 		(effects
 			(font
@@
 		(shape input)
 		(at 372.11 119.38 180)
-		(fields_autoplaced yes)
 		(effects
 			(font
@@
 		(shape input)
 		(at 154.94 129.54 180)
-		(fields_autoplaced yes)
 		(effects
 			(font
@@
 		(shape input)
 		(at 62.23 33.02 180)
-		(fields_autoplaced yes)
 		(effects
 			(font
@@
 		(shape input)
 		(at 236.22 125.73 180)
-		(fields_autoplaced yes)
 		(effects
 			(font
@@
 		(shape input)
 		(at 328.93 118.11 270)
-		(fields_autoplaced yes)
 		(effects
 			(font
@@
 		(shape input)
 		(at 477.52 104.14 0)
-		(fields_autoplaced yes)
 		(effects
 			(font
@@
 		(shape input)
 		(at 111.76 48.26 180)
-		(fields_autoplaced yes)
 		(effects
 			(font
@@
 		(shape input)
 		(at 298.45 104.14 270)
-		(fields_autoplaced yes)
 		(effects
 			(font
@@
 		(shape input)
 		(at 104.14 166.37 270)
-		(fields_autoplaced yes)
 		(effects
 			(font
@@
 		(shape input)
 		(at 48.26 109.22 180)
-		(fields_autoplaced yes)
 		(effects
 			(font
@@
 		(shape input)
 		(at 179.07 71.12 180)
-		(fields_autoplaced yes)
 		(effects
 			(font
@@
 		(shape input)
 		(at 86.36 166.37 270)
-		(fields_autoplaced yes)
 		(effects
 			(font
@@
 		(shape input)
 		(at 241.3 62.23 180)
-		(fields_autoplaced yes)
 		(effects
 			(font
@@
 		(shape input)
 		(at 403.86 125.73 180)
-		(fields_autoplaced yes)
 		(effects
 			(font
@@
 		(shape input)
 		(at 114.3 60.96 180)
-		(fields_autoplaced yes)
 		(effects
 			(font
@@
 		(shape input)
 		(at 50.8 137.16 180)
-		(fields_autoplaced yes)
 		(effects
 			(font
@@
 		(shape input)
 		(at 109.22 121.92 270)
-		(fields_autoplaced yes)
 		(effects
 			(font
@@
 			)
 		)
-		(property "Datasheet" "http://www.ti.com/lit/ds/symlink/uc2525b.pdf"
+		(property "Datasheet" "https://static.chipdip.ru/lib/877/DOC003877016.pdf"
 			(at 143.51 92.71 0)
 			(effects
@@
 			)
 		)
-		(property "Value" "SM6T30CA"
+		(property "Value" "SMAJ5.0CA-TR"
 			(at 69.85 132.0799 90)
 			(effects
@@
 		(in_bom yes)
 		(on_board yes)
-		(dnp no)
+		(dnp yes)
 		(property "Reference" "C35"
 			(at 111.76 160.02 0)
@@
 			)
 		)
-		(property "Value" "220"
+		(property "Value" "200"
 			(at 44.45 123.19 90)
 			(effects
@@
 			)
 		)
-		(property "Value" "1 uF"
-			(at 201.93 91.44 0)
+		(property "Value" "47 nF .... 120 nF *"
+			(at 209.55 91.44 0)
 			(effects
 				(font
@@
 			)
 		)
+		(property "Actual" "100 nF"
+			(at 203.962 92.964 0)
+			(effects
+				(font
+					(size 1.27 1.27)
+				)
+				(hide yes)
+			)
+		)
 		(pin "1"
 		)
@@
 			)
 		)
-		(property "Value" "4K7"
+		(property "Value" "1K2"
 			(at 90.17 162.56 0)
 			(effects
@@
 		(in_bom yes)
 		(on_board yes)
-		(dnp no)
+		(dnp yes)
 		(property "Reference" "C50"
 			(at 398.78 137.16 0)
