File: schematics/supply-uv/pwrcontrol.kicad_sch (KiCad schematic)
At the start: 35 parts, among them J5 USBASP, J6 JST XH B3B, J7 Conn_01x03_Pin, Q12 IRLML0030, Q13 IRLML0030, SW1 SW_Push, U19 TL431DBZ, U20 ATtiny1616-M, U21 ISO1540

Commit message: Board#1 schematics rewrited
Parts:
- added TP31: VSYS_GND, Library:TestPoint_Plated_Hole_D1.0mm, symbol Connector:TestPoint
- renumbered C69 to C68, C70 to C69, C68 to C70, D15 to D17, D16 to D18, D17 to D19, D18 to D20, J5 to J6, J6 to J7, J7 to J8, TP14 to TP32, TP15 to TP33, TP16 to TP34, TP17 to TP35, TP18 to TP36, TP19 to TP37, TP20 to TP38
Connections:
- net IS_ONOFF_BUTTON_PRESSED: now also U20.5 (PA4)
- net VSYS_PWR_GND: now also TP31.1
- no-connect marks 10 -> 9
Changed lines of the file:
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@@
 	)
 	(no_connect
-		(at 144.78 106.68)
-	)
-	(no_connect
 		(at 144.78 101.6)
 	)
@@
 	(wire
 		(pts
+			(xy 144.78 106.68) (xy 149.86 106.68)
+		)
+		(stroke
+			(width 0)
+			(type default)
+		)
+	)
+	(wire
+		(pts
 			(xy 486.41 121.92) (xy 486.41 124.46)
 		)
@@
 	(wire
 		(pts
+			(xy 83.82 223.52) (xy 88.9 223.52)
+		)
+		(stroke
+			(width 0)
+			(type default)
+		)
+	)
+	(wire
+		(pts
 			(xy 359.41 143.51) (xy 359.41 138.43)
 		)
@@
 		)
 	)
+	(label "IS_ONOFF_BUTTON_PRESSED"
+		(at 149.86 106.68 0)
+		(fields_autoplaced yes)
+		(effects
+			(font
+				(size 1.27 1.27)
+			)
+			(justify left bottom)
+		)
+	)
 	(label "POWER_OUTPUT_OVERLOADED_LED"
 		(at 107.95 124.46 180)
@@
 		)
 	)
+	(hierarchical_label "VSYS_PWR_GND"
+		(shape input)
+		(at 83.82 223.52 180)
+		(fields_autoplaced yes)
+		(effects
+			(font
+				(size 1.27 1.27)
+			)
+			(justify right)
+		)
+	)
 	(hierarchical_label "VSYS_GND"
 		(shape input)
@@
 		(dnp no)
 		(fields_autoplaced yes)
-		(property "Reference" "TP17"
+		(property "Reference" "TP35"
 			(at 222.25 109.728 0)
 			(effects
@@
 			(project "supply-uv"
 				(path "/ef40850c-d0bf-4cba-961b-9aba418f8e73/8f5c41f8-d5bb-4869-a96f-64e58008be54"
-					(reference "TP17")
+					(reference "TP35")
 					(unit 1)
 				)
@@
 		(dnp no)
 		(fields_autoplaced yes)
-		(property "Reference" "TP20"
+		(property "Reference" "TP38"
 			(at 521.97 105.918 0)
 			(effects
@@
 			(project "supply-uv"
 				(path "/ef40850c-d0bf-4cba-961b-9aba418f8e73/8f5c41f8-d5bb-4869-a96f-64e58008be54"
-					(reference "TP20")
+					(reference "TP38")
 					(unit 1)
 				)
@@
 		(dnp no)
 		(fields_autoplaced yes)
-		(property "Reference" "D18"
+		(property "Reference" "D20"
 			(at 502.92 88.9 0)
 			(effects
@@
 			(project "supply-uv"
 				(path "/ef40850c-d0bf-4cba-961b-9aba418f8e73/8f5c41f8-d5bb-4869-a96f-64e58008be54"
-					(reference "D18")
+					(reference "D20")
 					(unit 1)
 				)
@@
 		(dnp no)
 		(fields_autoplaced yes)
-		(property "Reference" "TP14"
+		(property "Reference" "TP32"
 			(at 222.25 77.9779 0)
 			(effects
@@
 			(project "supply-uv"
 				(path "/ef40850c-d0bf-4cba-961b-9aba418f8e73/8f5c41f8-d5bb-4869-a96f-64e58008be54"
-					(reference "TP14")
+					(reference "TP32")
 					(unit 1)
 				)
@@
 		(dnp no)
 		(fields_autoplaced yes)
-		(property "Reference" "TP15"
+		(property "Reference" "TP33"
 			(at 222.25 89.408 0)
 			(effects
@@
 			(project "supply-uv"
 				(path "/ef40850c-d0bf-4cba-961b-9aba418f8e73/8f5c41f8-d5bb-4869-a96f-64e58008be54"
-					(reference "TP15")
+					(reference "TP33")
 					(unit 1)
 				)
@@
 		(dnp no)
 		(fields_autoplaced yes)
-		(property "Reference" "TP18"
+		(property "Reference" "TP36"
 			(at 491.49 88.138 0)
 			(effects
@@
 			(project "supply-uv"
 				(path "/ef40850c-d0bf-4cba-961b-9aba418f8e73/8f5c41f8-d5bb-4869-a96f-64e58008be54"
-					(reference "TP18")
+					(reference "TP36")
 					(unit 1)
 				)
@@
 		(dnp no)
 		(fields_autoplaced yes)
-		(property "Reference" "TP16"
+		(property "Reference" "TP34"
 			(at 222.25 99.568 0)
 			(effects
@@
 			(project "supply-uv"
 				(path "/ef40850c-d0bf-4cba-961b-9aba418f8e73/8f5c41f8-d5bb-4869-a96f-64e58008be54"
-					(reference "TP16")
+					(reference "TP34")
 					(unit 1)
 				)
@@
 		(dnp no)
 		(fields_autoplaced yes)
-		(property "Reference" "J6"
+		(property "Reference" "J7"
 			(at 300.99 129.54 0)
 			(effects
@@
 			(project "supply-uv"
 				(path "/ef40850c-d0bf-4cba-961b-9aba418f8e73/8f5c41f8-d5bb-4869-a96f-64e58008be54"
-					(reference "J6")
+					(reference "J7")
 					(unit 1)
 				)
@@
 	)
 	(symbol
+		(lib_id "Connector:TestPoint")
+		(at 88.9 223.52 0)
+		(unit 1)
+		(exclude_from_sim no)
+		(in_bom yes)
+		(on_board yes)
+		(dnp no)
+		(fields_autoplaced yes)
+		(property "Reference" "TP31"
+			(at 91.44 218.9479 0)
+			(effects
+				(font
+					(size 1.27 1.27)
+				)
+				(justify left)
+			)
+		)
+		(property "Value" "VSYS_GND"
+			(at 91.44 221.4879 0)
+			(effects
+				(font
+					(size 1.27 1.27)
+				)
+				(justify left)
+			)
+		)
+		(property "Footprint" "Library:TestPoint_Plated_Hole_D1.0mm"
+			(at 93.98 223.52 0)
+			(effects
+				(font
+					(size 1.27 1.27)
+				)
+				(hide yes)
+			)
+		)
+		(property "Datasheet" "~"
+			(at 93.98 223.52 0)
+			(effects
+				(font
+					(size 1.27 1.27)
+				)
+				(hide yes)
+			)
+		)
+		(property "Description" "test point"
+			(at 88.9 223.52 0)
+			(effects
+				(font
+					(size 1.27 1.27)
+				)
+				(hide yes)
+			)
+		)
+		(pin "1"
+		)
+		(instances
+			(project "supply-uv"
+				(path "/ef40850c-d0bf-4cba-961b-9aba418f8e73/8f5c41f8-d5bb-4869-a96f-64e58008be54"
+					(reference "TP31")
+					(unit 1)
+				)
+			)
+		)
+	)
+	(symbol
 		(lib_id "Connector:Conn_01x03_Pin")
 		(at 322.58 130.81 0)
@@
 		(dnp no)
 		(fields_autoplaced yes)
-		(property "Reference" "J7"
+		(property "Reference" "J8"
 			(at 323.215 123.19 0)
 			(effects
@@
 			(project "supply-uv"
 				(path "/ef40850c-d0bf-4cba-961b-9aba418f8e73/8f5c41f8-d5bb-4869-a96f-64e58008be54"
-					(reference "J7")
+					(reference "J8")
 					(unit 1)
 				)
@@
 		(dnp no)
 		(fields_autoplaced yes)
-		(property "Reference" "J5"
+		(property "Reference" "J6"
 			(at 223.52 29.21 0)
 			(effects
@@
 			(project "supply-uv"
 				(path "/ef40850c-d0bf-4cba-961b-9aba418f8e73/8f5c41f8-d5bb-4869-a96f-64e58008be54"
-					(reference "J5")
+					(reference "J6")
 					(unit 1)
 				)
@@
 		(dnp no)
 		(fields_autoplaced yes)
-		(property "Reference" "C69"
+		(property "Reference" "C68"
 			(at 171.45 223.52 0)
 			(effects
@@
 			(project "supply-uv"
 				(path "/ef40850c-d0bf-4cba-961b-9aba418f8e73/8f5c41f8-d5bb-4869-a96f-64e58008be54"
-					(reference "C69")
+					(reference "C68")
 					(unit 1)
 				)
@@
 		(dnp no)
 		(fields_autoplaced yes)
-		(property "Reference" "C68"
+		(property "Reference" "C70"
 			(at 476.25 97.7899 0)
 			(effects
@@
 			(project "supply-uv"
 				(path "/ef40850c-d0bf-4cba-961b-9aba418f8e73/8f5c41f8-d5bb-4869-a96f-64e58008be54"
-					(reference "C68")
+					(reference "C70")
 					(unit 1)
 				)
@@
 		(dnp no)
 		(fields_autoplaced yes)
-		(property "Reference" "D16"
+		(property "Reference" "D18"
 			(at 363.22 134.9375 90)
 			(effects
@@
 			(project "supply-uv"
 				(path "/ef40850c-d0bf-4cba-961b-9aba418f8e73/8f5c41f8-d5bb-4869-a96f-64e58008be54"
-					(reference "D16")
+					(reference "D18")
 					(unit 1)
 				)
@@
 		(dnp no)
 		(fields_autoplaced yes)
-		(property "Reference" "TP19"
+		(property "Reference" "TP37"
 			(at 491.49 116.078 0)
 			(effects
@@
 			(project "supply-uv"
 				(path "/ef40850c-d0bf-4cba-961b-9aba418f8e73/8f5c41f8-d5bb-4869-a96f-64e58008be54"
-					(reference "TP19")
+					(reference "TP37")
 					(unit 1)
 				)
@@
 		(dnp no)
 		(fields_autoplaced yes)
-		(property "Reference" "D15"
+		(property "Reference" "D17"
 			(at 345.44 134.9375 90)
 			(effects
@@
 			(project "supply-uv"
 				(path "/ef40850c-d0bf-4cba-961b-9aba418f8e73/8f5c41f8-d5bb-4869-a96f-64e58008be54"
-					(reference "D15")
+					(reference "D17")
 					(unit 1)
 				)
@@
 		(dnp no)
 		(fields_autoplaced yes)
-		(property "Reference" "D17"
+		(property "Reference" "D19"
 			(at 501.65 116.84 0)
 			(effects
@@
 			(project "supply-uv"
 				(path "/ef40850c-d0bf-4cba-961b-9aba418f8e73/8f5c41f8-d5bb-4869-a96f-64e58008be54"
-					(reference "D17")
+					(reference "D19")
 					(unit 1)
 				)
@@
 		(dnp no)
 		(fields_autoplaced yes)
-		(property "Reference" "C70"
+		(property "Reference" "C69"
 			(at 194.31 223.52 0)
 			(effects
@@
 			(project "supply-uv"
 				(path "/ef40850c-d0bf-4cba-961b-9aba418f8e73/8f5c41f8-d5bb-4869-a96f-64e58008be54"
-					(reference "C70")
+					(reference "C69")
 					(unit 1)
 				)

Commit message: added some protection logic
Parts:
- removed C68, C69: 100 nF, Capacitor_SMD:C_0603_1608Metric, symbol Device:C
- removed U21: ISO1540, Package_SO:SOIC-8_3.9x4.9mm_P1.27mm, symbol Isolator:ISO1540
- renumbered C65 to C70, C66 to C71, C67 to C72, C70 to C73, D17 to D22, D18 to D23, D19 to D24, D20 to D25, Q12 to Q13, Q13 to Q14, R60 to R66, R61 to R67, R62 to R68, R63 to R69, R64 to R70, R65 to R71, R66 to R72, R67 to R73, R68 to R74, U19 to U21, U20 to U22
Connections:
- net VSYS_PWR renamed VSYS_PWR_VCC

Commit message: First board routing completed. I will review it few days later and maybe optimize something, but base worki done
Parts:
- renumbered C70 to C72, C71 to C73, C72 to C74, C73 to C75, R66 to R68, R67 to R69, R68 to R70, R69 to R71, R70 to R72, R71 to R73, R72 to R74, R73 to R75, R74 to R76, TP31 to TP27, TP32 to TP28, TP33 to TP29, TP34 to TP30, TP35 to TP31, TP36 to TP32, TP37 to TP33, TP38 to TP34
Changed lines of the file:
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@@
 		(dnp no)
 		(fields_autoplaced yes)
-		(property "Reference" "TP35"
+		(property "Reference" "TP31"
 			(at 222.25 109.728 0)
 			(effects
@@
 			(project "supply-uv"
 				(path "/ef40850c-d0bf-4cba-961b-9aba418f8e73/8f5c41f8-d5bb-4869-a96f-64e58008be54"
-					(reference "TP35")
+					(reference "TP31")
 					(unit 1)
 				)
@@
 		(dnp no)
 		(fields_autoplaced yes)
-		(property "Reference" "TP38"
+		(property "Reference" "TP34"
 			(at 521.97 105.918 0)
 			(effects
@@
 			(project "supply-uv"
 				(path "/ef40850c-d0bf-4cba-961b-9aba418f8e73/8f5c41f8-d5bb-4869-a96f-64e58008be54"
-					(reference "TP38")
+					(reference "TP34")
 					(unit 1)
 				)
@@
 		(dnp no)
 		(fields_autoplaced yes)
-		(property "Reference" "TP32"
+		(property "Reference" "TP28"
 			(at 222.25 77.9779 0)
 			(effects
@@
 			(project "supply-uv"
 				(path "/ef40850c-d0bf-4cba-961b-9aba418f8e73/8f5c41f8-d5bb-4869-a96f-64e58008be54"
-					(reference "TP32")
+					(reference "TP28")
 					(unit 1)
 				)
@@
 		(dnp no)
 		(fields_autoplaced yes)
-		(property "Reference" "R69"
+		(property "Reference" "R71"
 			(at 227.33 147.3199 0)
 			(effects
@@
 			(project "supply-uv"
 				(path "/ef40850c-d0bf-4cba-961b-9aba418f8e73/8f5c41f8-d5bb-4869-a96f-64e58008be54"
-					(reference "R69")
+					(reference "R71")
 					(unit 1)
 				)
@@
 		(dnp no)
 		(fields_autoplaced yes)
-		(property "Reference" "C70"
+		(property "Reference" "C72"
 			(at 99.06 91.44 0)
 			(effects
@@
 			(project "supply-uv"
 				(path "/ef40850c-d0bf-4cba-961b-9aba418f8e73/8f5c41f8-d5bb-4869-a96f-64e58008be54"
-					(reference "C70")
+					(reference "C72")
 					(unit 1)
 				)
@@
 		(dnp no)
 		(fields_autoplaced yes)
-		(property "Reference" "R73"
+		(property "Reference" "R75"
 			(at 488.95 127 0)
 			(effects
@@
 			(project "supply-uv"
 				(path "/ef40850c-d0bf-4cba-961b-9aba418f8e73/8f5c41f8-d5bb-4869-a96f-64e58008be54"
-					(reference "R73")
+					(reference "R75")
 					(unit 1)
 				)
@@
 		(dnp no)
 		(fields_autoplaced yes)
-		(property "Reference" "TP33"
+		(property "Reference" "TP29"
 			(at 222.25 89.408 0)
 			(effects
@@
 			(project "supply-uv"
 				(path "/ef40850c-d0bf-4cba-961b-9aba418f8e73/8f5c41f8-d5bb-4869-a96f-64e58008be54"
-					(reference "TP33")
+					(reference "TP29")
 					(unit 1)
 				)
@@
 		(dnp no)
 		(fields_autoplaced yes)
-		(property "Reference" "R66"
+		(property "Reference" "R68"
 			(at 72.39 149.86 90)
 			(effects
@@
 			(project "supply-uv"
 				(path "/ef40850c-d0bf-4cba-961b-9aba418f8e73/8f5c41f8-d5bb-4869-a96f-64e58008be54"
-					(reference "R66")
+					(reference "R68")
 					(unit 1)
 				)
@@
 		(dnp no)
 		(fields_autoplaced yes)
-		(property "Reference" "TP36"
+		(property "Reference" "TP32"
 			(at 491.49 88.138 0)
 			(effects
@@
 			(project "supply-uv"
 				(path "/ef40850c-d0bf-4cba-961b-9aba418f8e73/8f5c41f8-d5bb-4869-a96f-64e58008be54"
-					(reference "TP36")
+					(reference "TP32")
 					(unit 1)
 				)
@@
 		(dnp no)
 		(fields_autoplaced yes)
-		(property "Reference" "TP34"
+		(property "Reference" "TP30"
 			(at 222.25 99.568 0)
 			(effects
@@
 			(project "supply-uv"
 				(path "/ef40850c-d0bf-4cba-961b-9aba418f8e73/8f5c41f8-d5bb-4869-a96f-64e58008be54"
-					(reference "TP34")
+					(reference "TP30")
 					(unit 1)
 				)
@@
 		(dnp no)
 		(fields_autoplaced yes)
-		(property "Reference" "R70"
+		(property "Reference" "R72"
 			(at 279.4 165.1 0)
 			(effects
@@
 			(project "supply-uv"
 				(path "/ef40850c-d0bf-4cba-961b-9aba418f8e73/8f5c41f8-d5bb-4869-a96f-64e58008be54"
-					(reference "R70")
+					(reference "R72")
 					(unit 1)
 				)
@@
 		(dnp no)
 		(fields_autoplaced yes)
-		(property "Reference" "TP31"
+		(property "Reference" "TP27"
 			(at 91.44 218.9479 0)
 			(effects
@@
 			(project "supply-uv"
 				(path "/ef40850c-d0bf-4cba-961b-9aba418f8e73/8f5c41f8-d5bb-4869-a96f-64e58008be54"
-					(reference "TP31")
+					(reference "TP27")
 					(unit 1)
 				)
@@
 		(dnp no)
 		(fields_autoplaced yes)
-		(property "Reference" "R68"
+		(property "Reference" "R70"
 			(at 215.9 162.56 0)
 			(effects
@@
 			(project "supply-uv"
 				(path "/ef40850c-d0bf-4cba-961b-9aba418f8e73/8f5c41f8-d5bb-4869-a96f-64e58008be54"
-					(reference "R68")
+					(reference "R70")
 					(unit 1)
 				)
@@
 		(dnp no)
 		(fields_autoplaced yes)
-		(property "Reference" "C71"
+		(property "Reference" "C73"
 			(at 105.41 165.0999 0)
 			(effects
@@
 			(project "supply-uv"
 				(path "/ef40850c-d0bf-4cba-961b-9aba418f8e73/8f5c41f8-d5bb-4869-a96f-64e58008be54"
-					(reference "C71")
+					(reference "C73")
 					(unit 1)
 				)
@@
 		(dnp no)
 		(fields_autoplaced yes)
-		(property "Reference" "C73"
+		(property "Reference" "C75"
 			(at 476.25 97.7899 0)
 			(effects
@@
 			(project "supply-uv"
 				(path "/ef40850c-d0bf-4cba-961b-9aba418f8e73/8f5c41f8-d5bb-4869-a96f-64e58008be54"
-					(reference "C73")
+					(reference "C75")
 					(unit 1)
 				)
@@
 		(dnp no)
 		(fields_autoplaced yes)
-		(property "Reference" "C72"
+		(property "Reference" "C74"
 			(at 154.94 76.2 0)
 			(effects
@@
 			(project "supply-uv"
 				(path "/ef40850c-d0bf-4cba-961b-9aba418f8e73/8f5c41f8-d5bb-4869-a96f-64e58008be54"
-					(reference "C72")
+					(reference "C74")
 					(unit 1)
 				)
@@
 		(dnp no)
 		(fields_autoplaced yes)
-		(property "Reference" "R74"
+		(property "Reference" "R76"
 			(at 521.97 116.84 0)
 			(effects
@@
 			(project "supply-uv"
 				(path "/ef40850c-d0bf-4cba-961b-9aba418f8e73/8f5c41f8-d5bb-4869-a96f-64e58008be54"
-					(reference "R74")
+					(reference "R76")
 					(unit 1)
 				)
@@
 		(dnp no)
 		(fields_autoplaced yes)
-		(property "Reference" "R67"
+		(property "Reference" "R69"
 			(at 163.83 68.58 90)
 			(effects
@@
 			(project "supply-uv"
 				(path "/ef40850c-d0bf-4cba-961b-9aba418f8e73/8f5c41f8-d5bb-4869-a96f-64e58008be54"
-					(reference "R67")
+					(reference "R69")
 					(unit 1)
 				)
@@
 		(dnp no)
 		(fields_autoplaced yes)
-		(property "Reference" "R72"
+		(property "Reference" "R74"
 			(at 488.95 97.79 0)
 			(effects
@@
 			(project "supply-uv"
 				(path "/ef40850c-d0bf-4cba-961b-9aba418f8e73/8f5c41f8-d5bb-4869-a96f-64e58008be54"
-					(reference "R72")
+					(reference "R74")
 					(unit 1)
 				)
@@
 		(dnp no)
 		(fields_autoplaced yes)
-		(property "Reference" "TP37"
+		(property "Reference" "TP33"
 			(at 491.49 116.078 0)
 			(effects
@@
 			(project "supply-uv"
 				(path "/ef40850c-d0bf-4cba-961b-9aba418f8e73/8f5c41f8-d5bb-4869-a96f-64e58008be54"
-					(reference "TP37")
+					(reference "TP33")
 					(unit 1)
 				)
@@
 		(dnp no)
 		(fields_autoplaced yes)
-		(property "Reference" "R71"
+		(property "Reference" "R73"
 			(at 290.83 149.8599 0)
 			(effects
@@
 			(project "supply-uv"
 				(path "/ef40850c-d0bf-4cba-961b-9aba418f8e73/8f5c41f8-d5bb-4869-a96f-64e58008be54"
-					(reference "R71")
-					(unit 1)
-				)
+					(reference "R73")
+					(unit 1)
+				)

Commit message: Boards prepared to order
Parts:
- renumbered C72 to C73, C73 to C74, C74 to C75, C75 to C76, TP27 to TP29, TP28 to TP30, TP29 to TP31, TP30 to TP32, TP31 to TP33, TP32 to TP34, TP33 to TP35, TP34 to TP36
Changed lines of the file:
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@@
 		(dnp no)
 		(fields_autoplaced yes)
-		(property "Reference" "TP31"
+		(property "Reference" "TP33"
 			(at 222.25 109.728 0)
 			(effects
@@
 			(project "supply-uv"
 				(path "/ef40850c-d0bf-4cba-961b-9aba418f8e73/8f5c41f8-d5bb-4869-a96f-64e58008be54"
-					(reference "TP31")
+					(reference "TP33")
 					(unit 1)
 				)
@@
 		(dnp no)
 		(fields_autoplaced yes)
-		(property "Reference" "TP34"
+		(property "Reference" "TP36"
 			(at 521.97 105.918 0)
 			(effects
@@
 			(project "supply-uv"
 				(path "/ef40850c-d0bf-4cba-961b-9aba418f8e73/8f5c41f8-d5bb-4869-a96f-64e58008be54"
-					(reference "TP34")
+					(reference "TP36")
 					(unit 1)
 				)
@@
 		(dnp no)
 		(fields_autoplaced yes)
-		(property "Reference" "TP28"
+		(property "Reference" "TP30"
 			(at 222.25 77.9779 0)
 			(effects
@@
 			(project "supply-uv"
 				(path "/ef40850c-d0bf-4cba-961b-9aba418f8e73/8f5c41f8-d5bb-4869-a96f-64e58008be54"
-					(reference "TP28")
+					(reference "TP30")
 					(unit 1)
 				)
@@
 		(dnp no)
 		(fields_autoplaced yes)
-		(property "Reference" "C72"
+		(property "Reference" "C73"
 			(at 99.06 91.44 0)
 			(effects
@@
 			(project "supply-uv"
 				(path "/ef40850c-d0bf-4cba-961b-9aba418f8e73/8f5c41f8-d5bb-4869-a96f-64e58008be54"
-					(reference "C72")
+					(reference "C73")
 					(unit 1)
 				)
@@
 		(dnp no)
 		(fields_autoplaced yes)
-		(property "Reference" "TP29"
+		(property "Reference" "TP31"
 			(at 222.25 89.408 0)
 			(effects
@@
 			(project "supply-uv"
 				(path "/ef40850c-d0bf-4cba-961b-9aba418f8e73/8f5c41f8-d5bb-4869-a96f-64e58008be54"
-					(reference "TP29")
+					(reference "TP31")
 					(unit 1)
 				)
@@
 		(dnp no)
 		(fields_autoplaced yes)
-		(property "Reference" "TP32"
+		(property "Reference" "TP34"
 			(at 491.49 88.138 0)
 			(effects
@@
 			(project "supply-uv"
 				(path "/ef40850c-d0bf-4cba-961b-9aba418f8e73/8f5c41f8-d5bb-4869-a96f-64e58008be54"
-					(reference "TP32")
+					(reference "TP34")
 					(unit 1)
 				)
@@
 		(dnp no)
 		(fields_autoplaced yes)
-		(property "Reference" "TP30"
+		(property "Reference" "TP32"
 			(at 222.25 99.568 0)
 			(effects
@@
 			(project "supply-uv"
 				(path "/ef40850c-d0bf-4cba-961b-9aba418f8e73/8f5c41f8-d5bb-4869-a96f-64e58008be54"
-					(reference "TP30")
+					(reference "TP32")
 					(unit 1)
 				)
@@
 		(dnp no)
 		(fields_autoplaced yes)
-		(property "Reference" "TP27"
+		(property "Reference" "TP29"
 			(at 91.44 218.9479 0)
 			(effects
@@
 			(project "supply-uv"
 				(path "/ef40850c-d0bf-4cba-961b-9aba418f8e73/8f5c41f8-d5bb-4869-a96f-64e58008be54"
-					(reference "TP27")
+					(reference "TP29")
 					(unit 1)
 				)
@@
 		(dnp no)
 		(fields_autoplaced yes)
-		(property "Reference" "C73"
+		(property "Reference" "C74"
 			(at 105.41 165.0999 0)
 			(effects
@@
 			(project "supply-uv"
 				(path "/ef40850c-d0bf-4cba-961b-9aba418f8e73/8f5c41f8-d5bb-4869-a96f-64e58008be54"
-					(reference "C73")
+					(reference "C74")
 					(unit 1)
 				)
@@
 		(dnp no)
 		(fields_autoplaced yes)
-		(property "Reference" "C75"
+		(property "Reference" "C76"
 			(at 476.25 97.7899 0)
 			(effects
@@
 			(project "supply-uv"
 				(path "/ef40850c-d0bf-4cba-961b-9aba418f8e73/8f5c41f8-d5bb-4869-a96f-64e58008be54"
-					(reference "C75")
+					(reference "C76")
 					(unit 1)
 				)
@@
 		(dnp no)
 		(fields_autoplaced yes)
-		(property "Reference" "C74"
+		(property "Reference" "C75"
 			(at 154.94 76.2 0)
 			(effects
@@
 			(project "supply-uv"
 				(path "/ef40850c-d0bf-4cba-961b-9aba418f8e73/8f5c41f8-d5bb-4869-a96f-64e58008be54"
-					(reference "C74")
+					(reference "C75")
 					(unit 1)
 				)
@@
 		(dnp no)
 		(fields_autoplaced yes)
-		(property "Reference" "TP33"
+		(property "Reference" "TP35"
 			(at 491.49 116.078 0)
 			(effects
@@
 			(project "supply-uv"
 				(path "/ef40850c-d0bf-4cba-961b-9aba418f8e73/8f5c41f8-d5bb-4869-a96f-64e58008be54"
-					(reference "TP33")
-					(unit 1)
-				)
+					(reference "TP35")
+					(unit 1)
+				)
